File: board/evm/circuit/usb_dongle.sch (KiCad schematic (older format))
At the start: 1 part

Commit message: add lots of ICs
Parts:
- removed U?: STM32F405VGTx, LQFP100, symbol STM32F405VGTx
- added U?: nRF24LU1+, symbol nRF24LU1+
Changed lines of the file:
@@
 EELAYER 25 0
 EELAYER END
-$Descr A2 23386 16535
+$Descr A4 11693 8268
 encoding utf-8
-Sheet 2 8
+Sheet 7 8
 Title ""
 Date ""
@@
 $EndDescr
 $Comp
-L STM32F405VGTx U?
-U 1 1 5753F449
-P 9650 6400
-F 0 "U?" H 5350 9225 50  0000 L BNN
-F 1 "STM32F405VGTx" H 13950 9225 50  0000 R BNN
-F 2 "LQFP100" H 13950 9175 50  0000 R TNN
-F 3 "" H 9650 6400 50  0000 C CNN
-	1    9650 6400
+L nRF24LU1+ U?
+U 1 1 5754763F
+P 3500 2850
+F 0 "U?" H 3500 2850 60  0000 C CNN
+F 1 "nRF24LU1+" H 3500 2750 60  0000 C CNN
+F 2 "" H 3500 2850 60  0000 C CNN
+F 3 "" H 3500 2850 60  0000 C CNN
+	1    3500 2850
 	1    0    0    -1
 $EndComp
