File: board/evm/circuit/usb_dongle.sch (KiCad schematic (older format))
At the start: 24 parts, among them J3 TagConnect, P2 USB_A, U9 nRF24LU1+, Y3 CRYSTAL_SMT

Commit message: working on footprint
Parts:
- C28: footprint (none) -> Capacitors_SMD:C_0805
- C29, C30, C31, C32, C33, C34, C35: footprint (none) -> Capacitors_SMD:C_0402
- D10: footprint (none) -> LEDs:LED_0805
- R10, R11, R12, R13, R14, R8, R9: footprint (none) -> Resistors_SMD:R_0402
- U9: footprint (none) -> Housings_DFN_QFN:QFN-32-1EP_5x5mm_Pitch0.5mm
Changed lines of the file:
@@
 F 0 "U9" H 5650 3100 60  0000 C CNN
 F 1 "nRF24LU1+" H 5650 3000 60  0000 C CNN
-F 2 "" H 5650 3100 60  0000 C CNN
+F 2 "Housings_DFN_QFN:QFN-32-1EP_5x5mm_Pitch0.5mm" H 5650 3100 60  0001 C CNN
 F 3 "" H 5650 3100 60  0000 C CNN
 	1    5650 3100
@@
 F 0 "P2" H 3700 2800 50  0000 C CNN
 F 1 "USB_A" H 3450 3200 50  0000 C CNN
-F 2 "" V 3450 2900 50  0000 C CNN
+F 2 "" V 3450 2900 50  0001 C CNN
 F 3 "" V 3450 2900 50  0000 C CNN
 	1    3500 3000
@@
 F 0 "R8" V 4230 3000 50  0000 C CNN
 F 1 "R22" V 4150 3000 50  0000 C CNN
-F 2 "" V 4080 3000 50  0000 C CNN
+F 2 "Resistors_SMD:R_0402" V 4080 3000 50  0001 C CNN
 F 3 "" H 4150 3000 50  0000 C CNN
 	1    4150 3000
@@
 F 0 "R10" V 4530 3100 50  0000 C CNN
 F 1 "R22" V 4450 3100 50  0000 C CNN
-F 2 "" V 4380 3100 50  0000 C CNN
+F 2 "Resistors_SMD:R_0402" V 4380 3100 50  0001 C CNN
 F 3 "" H 4450 3100 50  0000 C CNN
 	1    4450 3100
@@
 F 0 "C28" H 4460 2770 50  0000 L CNN
 F 1 "10uF" H 4460 2620 50  0000 L CNN
-F 2 "" H 4450 2700 50  0000 C CNN
+F 2 "Capacitors_SMD:C_0805" H 4450 2700 50  0001 C CNN
 F 3 "" H 4450 2700 50  0000 C CNN
 	1    4450 2700
@@
 F 0 "R9" V 4280 2800 50  0000 C CNN
 F 1 "R10" V 4200 2800 50  0000 C CNN
-F 2 "" V 4130 2800 50  0000 C CNN
+F 2 "Resistors_SMD:R_0402" V 4130 2800 50  0001 C CNN
 F 3 "" H 4200 2800 50  0000 C CNN
 	1    4200 2800
@@
 F 0 "R11" V 4680 3450 50  0000 C CNN
 F 1 "R10K" V 4600 3450 50  0000 C CNN
-F 2 "" V 4530 3450 50  0000 C CNN
+F 2 "Resistors_SMD:R_0402" V 4530 3450 50  0001 C CNN
 F 3 "" H 4600 3450 50  0000 C CNN
 	1    4600 3450
@@
 F 0 "R12" V 4830 3550 50  0000 C CNN
 F 1 "R10K" V 4750 3550 50  0000 C CNN
-F 2 "" V 4680 3550 50  0000 C CNN
+F 2 "Resistors_SMD:R_0402" V 4680 3550 50  0001 C CNN
 F 3 "" H 4750 3550 50  0000 C CNN
 	1    4750 3550
@@
 F 0 "C29" H 5110 4320 50  0000 L CNN
 F 1 "10nF" H 5110 4170 50  0000 L CNN
-F 2 "" H 5100 4250 50  0000 C CNN
+F 2 "Capacitors_SMD:C_0402" H 5100 4250 50  0001 C CNN
 F 3 "" H 5100 4250 50  0000 C CNN
 	1    5100 4250
@@
 F 0 "Y3" H 5100 1900 60  0000 C CNN
 F 1 "CRYSTAL_SMT" H 5100 1800 60  0000 C CNN
-F 2 "" H 5100 1600 60  0000 C CNN
+F 2 "" H 5100 1600 60  0001 C CNN
 F 3 "" H 5100 1600 60  0000 C CNN
 	1    5100 1600
@@
 F 0 "C30" H 5760 1420 50  0000 L CNN
 F 1 "33nF" H 5760 1270 50  0000 L CNN
-F 2 "" H 5750 1350 50  0000 C CNN
+F 2 "Capacitors_SMD:C_0402" H 5750 1350 50  0001 C CNN
 F 3 "" H 5750 1350 50  0000 C CNN
 	1    5750 1350
@@
 F 0 "C31" H 5960 1570 50  0000 L CNN
 F 1 "33nF" H 5960 1420 50  0000 L CNN
-F 2 "" H 5950 1500 50  0000 C CNN
+F 2 "Capacitors_SMD:C_0402" H 5950 1500 50  0001 C CNN
 F 3 "" H 5950 1500 50  0000 C CNN
 	1    5950 1500
@@
 F 0 "R13" V 6180 1700 50  0000 C CNN
 F 1 "R22K" V 6100 1700 50  0000 C CNN
-F 2 "" V 6030 1700 50  0000 C CNN
+F 2 "Resistors_SMD:R_0402" V 6030 1700 50  0001 C CNN
 F 3 "" H 6100 1700 50  0000 C CNN
 	1    6100 1700
@@
 F 0 "L7" H 7630 2990 50  0000 L CNN
 F 1 "6.8nH" H 7630 2910 50  0000 L CNN
-F 2 "" H 7600 2950 50  0000 C CNN
+F 2 "" H 7600 2950 50  0001 C CNN
 F 3 "" H 7600 2950 50  0000 C CNN
 	1    7600 2950
@@
 F 0 "L8" V 7850 2550 50  0000 L CNN
 F 1 "4.7nH" V 8050 2600 50  0000 L CNN
-F 2 "" H 7950 2650 50  0000 C CNN
+F 2 "" H 7950 2650 50  0001 C CNN
 F 3 "" H 7950 2650 50  0000 C CNN
 	1    7950 2650
@@
 F 0 "L9" V 7850 3050 50  0000 L CNN
 F 1 "6.8nH" V 8050 3100 50  0000 L CNN
-F 2 "" H 7950 3150 50  0000 C CNN
+F 2 "" H 7950 3150 50  0001 C CNN
 F 3 "" H 7950 3150 50  0000 C CNN
 	1    7950 3150
@@
 F 0 "C32" H 7710 3670 50  0000 L CNN
 F 1 "2.2nF" H 7710 3520 50  0000 L CNN
-F 2 "" H 7700 3600 50  0000 C CNN
+F 2 "Capacitors_SMD:C_0402" H 7700 3600 50  0001 C CNN
 F 3 "" H 7700 3600 50  0000 C CNN
 	1    7700 3600
@@
 F 0 "C33" H 8110 3670 50  0000 L CNN
 F 1 "NA" H 8110 3520 50  0000 L CNN
-F 2 "" H 8100 3600 50  0000 C CNN
+F 2 "Capacitors_SMD:C_0402" H 8100 3600 50  0001 C CNN
 F 3 "" H 8100 3600 50  0000 C CNN
 	1    8100 3600
@@
 F 0 "C34" H 8410 2720 50  0000 L CNN
 F 1 "1.2pF" H 8410 2570 50  0000 L CNN
-F 2 "" H 8400 2650 50  0000 C CNN
+F 2 "Capacitors_SMD:C_0402" H 8400 2650 50  0001 C CNN
 F 3 "" H 8400 2650 50  0000 C CNN
 	1    8400 2650
@@
 F 0 "C35" H 8710 3020 50  0000 L CNN
 F 1 "1.0pF" H 8710 2870 50  0000 L CNN
-F 2 "" H 8700 2950 50  0000 C CNN
+F 2 "Capacitors_SMD:C_0402" H 8700 2950 50  0001 C CNN
 F 3 "" H 8700 2950 50  0000 C CNN
 	1    8700 2950
@@
 F 0 "E3" H 9100 2750 60  0000 C CNN
 F 1 "ANTPCB" H 9200 2500 60  0000 C CNN
-F 2 "" H 9200 2600 60  0000 C CNN
+F 2 "" H 9200 2600 60  0001 C CNN
 F 3 "" H 9200 2600 60  0000 C CNN
 	1    9200 2600
@@
 F 0 "R14" V 6330 4450 50  0000 C CNN
 F 1 "330" V 6250 4450 50  0000 C CNN
-F 2 "" V 6180 4450 50  0000 C CNN
+F 2 "Resistors_SMD:R_0402" V 6180 4450 50  0001 C CNN
 F 3 "" H 6250 4450 50  0000 C CNN
 	1    6250 4450
@@
 F 0 "D10" H 5900 4550 50  0000 C CNN
 F 1 "LED" H 5900 4350 50  0000 C CNN
-F 2 "" H 5900 4450 50  0000 C CNN
+F 2 "LEDs:LED_0805" H 5900 4450 50  0001 C CNN
 F 3 "" H 5900 4450 50  0000 C CNN
 	1    5900 4450
@@
 F 0 "J3" H 3000 4150 60  0000 C CNN
 F 1 "TagConnect" H 3500 4150 60  0000 C CNN
-F 2 "" H 3150 4350 60  0000 C CNN
+F 2 "" H 3150 4350 60  0001 C CNN
 F 3 "" H 3150 4350 60  0000 C CNN
 	1    3300 4300
