File: board/evm/circuit/baseboard.sch (KiCad schematic (older format))
At the start: 28 parts

Commit message: evm sch design finished
Changed lines of the file:
@@
 LIBS:contrib
 LIBS:valves
-LIBS:stm8
-LIBS:stm32
-LIBS:74xgxx
-LIBS:ac-dc
-LIBS:actel
 LIBS:Altera
-LIBS:analog_devices
-LIBS:battery_management
-LIBS:bbd
-LIBS:brooktre
-LIBS:cmos_ieee
-LIBS:dc-dc
-LIBS:diode
-LIBS:elec-unifil
-LIBS:ESD_Protection
-LIBS:ftdi
-LIBS:gennum
-LIBS:graphic
-LIBS:hc11
-LIBS:ir
-LIBS:Lattice
-LIBS:logo
-LIBS:maxim
-LIBS:microchip_dspic33dsc
-LIBS:microchip_pic10mcu
-LIBS:microchip_pic12mcu
-LIBS:microchip_pic16mcu
-LIBS:microchip_pic18mcu
-LIBS:microchip_pic32mcu
-LIBS:motor_drivers
-LIBS:msp430
-LIBS:nordicsemi
-LIBS:nxp_armmcu
-LIBS:onsemi
-LIBS:Oscillators
-LIBS:powerint
-LIBS:Power_Management
-LIBS:pspice
-LIBS:references
-LIBS:relays
-LIBS:rfcom
-LIBS:sensors
-LIBS:silabs
-LIBS:supertex
-LIBS:switches
-LIBS:transf
-LIBS:ttl_ieee
-LIBS:video
-LIBS:Worldsemi
-LIBS:Xicor
-LIBS:Zilog
+LIBS:my_kicad
 LIBS:oh-my-keyboard-cache
 EELAYER 25 0
@@
 $Descr A3 16535 11693
 encoding utf-8
-Sheet 3 11
+Sheet 13 12
 Title ""
 Date ""
@@
 U 1 1 57533436
 P 1900 1850
+AR Path="/576F1415/57533436" Ref="SW?"  Part="1"
+AR Path="/57532E7E/57533436" Ref="SW?"  Part="1"
 F 0 "SW?" H 2050 1960 50  0000 C CNN
 F 1 "SW_PUSH" H 1900 1770 50  0000 C CNN
@@
 U 1 1 57533459
 P 1900 2100
+AR Path="/576F1415/57533459" Ref="SW?"  Part="1"
+AR Path="/57532E7E/57533459" Ref="SW?"  Part="1"
 F 0 "SW?" H 2050 2210 50  0000 C CNN
 F 1 "SW_PUSH" H 1900 2020 50  0000 C CNN
@@
 U 1 1 5753348E
 P 1900 2350
+AR Path="/576F1415/5753348E" Ref="SW?"  Part="1"
+AR Path="/57532E7E/5753348E" Ref="SW?"  Part="1"
 F 0 "SW?" H 2050 2460 50  0000 C CNN
 F 1 "SW_PUSH" H 1900 2270 50  0000 C CNN
@@
 U 1 1 575334CD
 P 1900 2600
+AR Path="/576F1415/575334CD" Ref="SW?"  Part="1"
+AR Path="/57532E7E/575334CD" Ref="SW?"  Part="1"
 F 0 "SW?" H 2050 2710 50  0000 C CNN
 F 1 "SW_PUSH" H 1900 2520 50  0000 C CNN
@@
 U 1 1 575334E8
 P 1900 2850
+AR Path="/576F1415/575334E8" Ref="SW?"  Part="1"
+AR Path="/57532E7E/575334E8" Ref="SW?"  Part="1"
 F 0 "SW?" H 2050 2960 50  0000 C CNN
 F 1 "SW_PUSH" H 1900 2770 50  0000 C CNN
@@
 U 1 1 575335A3
 P 1900 3100
+AR Path="/576F1415/575335A3" Ref="SW?"  Part="1"
+AR Path="/57532E7E/575335A3" Ref="SW?"  Part="1"
 F 0 "SW?" H 2050 3210 50  0000 C CNN
 F 1 "SW_PUSH" H 1900 3020 50  0000 C CNN
@@
 U 1 1 575335EE
 P 1900 3350
+AR Path="/576F1415/575335EE" Ref="SW?"  Part="1"
+AR Path="/57532E7E/575335EE" Ref="SW?"  Part="1"
 F 0 "SW?" H 2050 3460 50  0000 C CNN
 F 1 "SW_PUSH" H 1900 3270 50  0000 C CNN
@@
 U 1 1 57533614
 P 1900 3600
+AR Path="/576F1415/57533614" Ref="SW?"  Part="1"
+AR Path="/57532E7E/57533614" Ref="SW?"  Part="1"
 F 0 "SW?" H 2050 3710 50  0000 C CNN
 F 1 "SW_PUSH" H 1900 3520 50  0000 C CNN
@@
 U 1 1 57533BD4
 P 5700 1600
+AR Path="/576F1415/57533BD4" Ref="D?"  Part="1"
+AR Path="/57532E7E/57533BD4" Ref="D?"  Part="1"
 F 0 "D?" H 5775 1950 50  0000 C CNN
 F 1 "LED_RABG" H 5725 1250 50  0000 C CNN
@@
 U 1 1 57533C2F
 P 5700 2400
+AR Path="/576F1415/57533C2F" Ref="D?"  Part="1"
+AR Path="/57532E7E/57533C2F" Ref="D?"  Part="1"
 F 0 "D?" H 5775 2750 50  0000 C CNN
 F 1 "LED_RABG" H 5725 2050 50  0000 C CNN
@@
 U 1 1 57533CEE
 P 5700 3200
+AR Path="/576F1415/57533CEE" Ref="D?"  Part="1"
+AR Path="/57532E7E/57533CEE" Ref="D?"  Part="1"
 F 0 "D?" H 5775 3550 50  0000 C CNN
 F 1 "LED_RABG" H 5725 2850 50  0000 C CNN
@@
 U 1 1 57533DB5
 P 5700 4000
+AR Path="/576F1415/57533DB5" Ref="D?"  Part="1"
+AR Path="/57532E7E/57533DB5" Ref="D?"  Part="1"
 F 0 "D?" H 5775 4350 50  0000 C CNN
 F 1 "LED_RABG" H 5725 3650 50  0000 C CNN
@@
 U 1 1 57533DF4
 P 5700 4800
+AR Path="/576F1415/57533DF4" Ref="D?"  Part="1"
+AR Path="/57532E7E/57533DF4" Ref="D?"  Part="1"
 F 0 "D?" H 5775 5150 50  0000 C CNN
 F 1 "LED_RABG" H 5725 4450 50  0000 C CNN
@@
 U 1 1 57533E27
 P 5700 5600
+AR Path="/576F1415/57533E27" Ref="D?"  Part="1"
+AR Path="/57532E7E/57533E27" Ref="D?"  Part="1"
 F 0 "D?" H 5775 5950 50  0000 C CNN
 F 1 "LED_RABG" H 5725 5250 50  0000 C CNN
@@
 U 1 1 57533E80
 P 5700 6400
+AR Path="/576F1415/57533E80" Ref="D?"  Part="1"
+AR Path="/57532E7E/57533E80" Ref="D?"  Part="1"
 F 0 "D?" H 5775 6750 50  0000 C CNN
 F 1 "LED_RABG" H 5725 6050 50  0000 C CNN
@@
 U 1 1 57533EB1
 P 5700 7200
+AR Path="/576F1415/57533EB1" Ref="D?"  Part="1"
+AR Path="/57532E7E/57533EB1" Ref="D?"  Part="1"
 F 0 "D?" H 5775 7550 50  0000 C CNN
 F 1 "LED_RABG" H 5725 6850 50  0000 C CNN
@@
 U 1 1 5753FD79
 P 1400 5200
+AR Path="/576F1415/5753FD79" Ref="#PWR?"  Part="1"
+AR Path="/57532E7E/5753FD79" Ref="#PWR?"  Part="1"
 F 0 "#PWR?" H 1400 5050 50  0001 C CNN
 F 1 "+3V3" H 1400 5340 50  0000 C CNN
@@
 U 1 1 5753FDB5
 P 1400 6000
+AR Path="/576F1415/5753FDB5" Ref="#PWR?"  Part="1"
+AR Path="/57532E7E/5753FDB5" Ref="#PWR?"  Part="1"
 F 0 "#PWR?" H 1400 5750 50  0001 C CNN
 F 1 "GND" H 1400 5850 50  0000 C CNN
@@
 U 1 1 57540218
 P 750 900
+AR Path="/576F1415/57540218" Ref="#PWR?"  Part="1"
+AR Path="/57532E7E/57540218" Ref="#PWR?"  Part="1"
 F 0 "#PWR?" H 750 750 50  0001 C CNN
 F 1 "+3V3" H 750 1040 50  0000 C CNN
@@
 U 1 1 5754024D
 P 750 1200
+AR Path="/576F1415/5754024D" Ref="R?"  Part="1"
+AR Path="/57532E7E/5754024D" Ref="R?"  Part="1"
 F 0 "R?" V 830 1200 50  0000 C CNN
 F 1 "R100" V 750 1200 50  0000 C CNN
@@
 U 1 1 57541C46
 P 2400 4100
+AR Path="/576F1415/57541C46" Ref="R?"  Part="1"
+AR Path="/57532E7E/57541C46" Ref="R?"  Part="1"
 F 0 "R?" V 2480 4100 50  0000 C CNN
 F 1 "R1K" V 2400 4100 50  0000 C CNN
@@
 U 1 1 57541D0C
 P 2400 4400
+AR Path="/576F1415/57541D0C" Ref="#PWR?"  Part="1"
+AR Path="/57532E7E/57541D0C" Ref="#PWR?"  Part="1"
 F 0 "#PWR?" H 2400 4150 50  0001 C CNN
 F 1 "GND" H 2400 4250 50  0000 C CNN
@@
 U 1 1 57542572
 P 5050 900
+AR Path="/576F1415/57542572" Ref="#PWR?"  Part="1"
+AR Path="/57532E7E/57542572" Ref="#PWR?"  Part="1"
 F 0 "#PWR?" H 5050 750 50  0001 C CNN
 F 1 "+3V3" H 5050 1040 50  0000 C CNN
@@
 U 1 1 57542EEF
 P 7150 1600
+AR Path="/576F1415/57542EEF" Ref="RP?"  Part="1"
+AR Path="/57532E7E/57542EEF" Ref="RP?"  Part="1"
 F 0 "RP?" H 7150 2050 50  0000 C CNN
 F 1 "R_1K" H 7150 1550 50  0000 C CNN
@@
 U 1 1 5754341A
 P 7700 2000
+AR Path="/576F1415/5754341A" Ref="RP?"  Part="1"
+AR Path="/57532E7E/5754341A" Ref="RP?"  Part="1"
 F 0 "RP?" H 7700 2450 50  0000 C CNN
 F 1 "R_1K" H 7700 1950 50  0000 C CNN
@@
 U 1 1 575436DE
 P 7150 4300
+AR Path="/576F1415/575436DE" Ref="RP?"  Part="1"
+AR Path="/57532E7E/575436DE" Ref="RP?"  Part="1"
 F 0 "RP?" H 7150 4750 50  0000 C CNN
 F 1 "R_1K" H 7150 4250 50  0000 C CNN
@@
 U 1 1 575436E4
 P 7700 4700
+AR Path="/576F1415/575436E4" Ref="RP?"  Part="1"
+AR Path="/57532E7E/575436E4" Ref="RP?"  Part="1"
 F 0 "RP?" H 7700 5150 50  0000 C CNN
 F 1 "R_1K" H 7700 4650 50  0000 C CNN
@@
 U 1 1 57543834
 P 7150 6650
+AR Path="/576F1415/57543834" Ref="RP?"  Part="1"
+AR Path="/57532E7E/57543834" Ref="RP?"  Part="1"
 F 0 "RP?" H 7150 7100 50  0000 C CNN
 F 1 "R_1K" H 7150 6600 50  0000 C CNN
@@
 U 1 1 5754383A
 P 7700 7050
+AR Path="/576F1415/5754383A" Ref="RP?"  Part="1"
+AR Path="/57532E7E/5754383A" Ref="RP?"  Part="1"
 F 0 "RP?" H 7700 7500 50  0000 C CNN
 F 1 "R_1K" H 7700 7000 50  0000 C CNN
@@
 U 1 1 57532E87
 P 3850 2900
+AR Path="/576F1415/57532E87" Ref="U?"  Part="1"
+AR Path="/57532E7E/57532E87" Ref="U?"  Part="1"
 F 0 "U?" H 4000 2850 50  0000 C CNN
 F 1 "74LS165" H 4000 2650 50  0000 C CNN
@@
 U 1 1 57551E52
 P 9650 1700
+AR Path="/576F1415/57551E52" Ref="U?"  Part="1"
+AR Path="/57532E7E/57551E52" Ref="U?"  Part="1"
 F 0 "U?" H 9800 2300 70  0000 C CNN
 F 1 "74HC595" H 9650 1100 70  0000 C CNN
@@
 U 1 1 57552B2B
 P 9650 4400
+AR Path="/576F1415/57552B2B" Ref="U?"  Part="1"
+AR Path="/57532E7E/57552B2B" Ref="U?"  Part="1"
 F 0 "U?" H 9800 5000 70  0000 C CNN
 F 1 "74HC595" H 9650 3800 70  0000 C CNN
@@
 U 1 1 57552CFC
 P 9650 6750
+AR Path="/576F1415/57552CFC" Ref="U?"  Part="1"
+AR Path="/57532E7E/57552CFC" Ref="U?"  Part="1"
 F 0 "U?" H 9800 7350 70  0000 C CNN
 F 1 "74HC595" H 9650 6150 70  0000 C CNN
@@
 	3150 2700 2550 2700
 Wire Wire Line
-	2550 2600 2550 2700
-Wire Wire Line
-	2200 2600 2550 2600
+	2550 2700 2550 2600
+Wire Wire Line
+	2550 2600 2200 2600
 Wire Wire Line
 	2200 2850 2550 2850
@@
 	3150 2900 2600 2900
 Wire Wire Line
-	2600 3100 2600 2900
-Wire Wire Line
-	2200 3100 2600 3100
+	2600 2900 2600 3100
+Wire Wire Line
+	2600 3100 2200 3100
 Wire Wire Line
 	3150 3000 2650 3000
 Wire Wire Line
-	2650 3350 2650 3000
-Wire Wire Line
-	2200 3350 2650 3350
+	2650 3000 2650 3350
+Wire Wire Line
+	2650 3350 2200 3350
 Wire Wire Line
 	2200 3600 2700 3600
@@
 U 1 1 5755C449
 P 1100 900
+AR Path="/576F1415/5755C449" Ref="#PWR?"  Part="1"
+AR Path="/57532E7E/5755C449" Ref="#PWR?"  Part="1"
 F 0 "#PWR?" H 1100 750 50  0001 C CNN
 F 1 "VCC" H 1100 1050 50  0000 C CNN
