File: board/evm/circuit/baseboard.sch (KiCad schematic (older format))
At the start: 28 parts

Commit message: working on drc
Parts:
- gave numbers to parts that had none: 28
Connections:
- no-connect marks 0 -> 1

Commit message: working on footprint
Parts:
- D1, D2, D3, D4, D5, D6, D7, D8: footprint (none) -> LEDs:LED_RGB_Getian_GT-P6PRGB4303
- R3, R4, RP1, RP2, RP3, RP4, RP5, RP6: footprint (none) -> Resistors_SMD:R_0402
- SW1, SW2, SW3, SW4, SW5, SW6, SW7, SW8: footprint (none) -> Buttons_Switches_SMD:SW_SPST_B3U-1000P
- U1, U2, U3, U4: footprint (none) -> Housings_SSOP:TSSOP-16_4.4x5mm_Pitch0.65mm
Changed lines of the file:
@@
 F 0 "SW1" H 2050 1960 50  0000 C CNN
 F 1 "SW_PUSH" H 1900 1770 50  0000 C CNN
-F 2 "" H 1900 1850 50  0000 C CNN
+F 2 "Buttons_Switches_SMD:SW_SPST_B3U-1000P" H 1900 1850 50  0001 C CNN
 F 3 "" H 1900 1850 50  0000 C CNN
 	1    1900 1850
@@
 F 0 "SW2" H 2050 2210 50  0000 C CNN
 F 1 "SW_PUSH" H 1900 2020 50  0000 C CNN
-F 2 "" H 1900 2100 50  0000 C CNN
+F 2 "Buttons_Switches_SMD:SW_SPST_B3U-1000P" H 1900 2100 50  0001 C CNN
 F 3 "" H 1900 2100 50  0000 C CNN
 	1    1900 2100
@@
 F 0 "SW3" H 2050 2460 50  0000 C CNN
 F 1 "SW_PUSH" H 1900 2270 50  0000 C CNN
-F 2 "" H 1900 2350 50  0000 C CNN
+F 2 "Buttons_Switches_SMD:SW_SPST_B3U-1000P" H 1900 2350 50  0001 C CNN
 F 3 "" H 1900 2350 50  0000 C CNN
 	1    1900 2350
@@
 F 0 "SW4" H 2050 2710 50  0000 C CNN
 F 1 "SW_PUSH" H 1900 2520 50  0000 C CNN
-F 2 "" H 1900 2600 50  0000 C CNN
+F 2 "Buttons_Switches_SMD:SW_SPST_B3U-1000P" H 1900 2600 50  0001 C CNN
 F 3 "" H 1900 2600 50  0000 C CNN
 	1    1900 2600
@@
 F 0 "SW5" H 2050 2960 50  0000 C CNN
 F 1 "SW_PUSH" H 1900 2770 50  0000 C CNN
-F 2 "" H 1900 2850 50  0000 C CNN
+F 2 "Buttons_Switches_SMD:SW_SPST_B3U-1000P" H 1900 2850 50  0001 C CNN
 F 3 "" H 1900 2850 50  0000 C CNN
 	1    1900 2850
@@
 F 0 "SW6" H 2050 3210 50  0000 C CNN
 F 1 "SW_PUSH" H 1900 3020 50  0000 C CNN
-F 2 "" H 1900 3100 50  0000 C CNN
+F 2 "Buttons_Switches_SMD:SW_SPST_B3U-1000P" H 1900 3100 50  0001 C CNN
 F 3 "" H 1900 3100 50  0000 C CNN
 	1    1900 3100
@@
 F 0 "SW7" H 2050 3460 50  0000 C CNN
 F 1 "SW_PUSH" H 1900 3270 50  0000 C CNN
-F 2 "" H 1900 3350 50  0000 C CNN
+F 2 "Buttons_Switches_SMD:SW_SPST_B3U-1000P" H 1900 3350 50  0001 C CNN
 F 3 "" H 1900 3350 50  0000 C CNN
 	1    1900 3350
@@
 F 0 "SW8" H 2050 3710 50  0000 C CNN
 F 1 "SW_PUSH" H 1900 3520 50  0000 C CNN
-F 2 "" H 1900 3600 50  0000 C CNN
+F 2 "Buttons_Switches_SMD:SW_SPST_B3U-1000P" H 1900 3600 50  0001 C CNN
 F 3 "" H 1900 3600 50  0000 C CNN
 	1    1900 3600
@@
 F 0 "D1" H 5775 1950 50  0000 C CNN
 F 1 "LED_RABG" H 5725 1250 50  0000 C CNN
-F 2 "" H 5650 1550 50  0000 C CNN
+F 2 "LEDs:LED_RGB_Getian_GT-P6PRGB4303" H 5650 1550 50  0001 C CNN
 F 3 "" H 5650 1550 50  0000 C CNN
 	1    5700 1600
@@
 F 0 "D2" H 5775 2750 50  0000 C CNN
 F 1 "LED_RABG" H 5725 2050 50  0000 C CNN
-F 2 "" H 5650 2350 50  0000 C CNN
+F 2 "LEDs:LED_RGB_Getian_GT-P6PRGB4303" H 5650 2350 50  0001 C CNN
 F 3 "" H 5650 2350 50  0000 C CNN
 	1    5700 2400
@@
 F 0 "D3" H 5775 3550 50  0000 C CNN
 F 1 "LED_RABG" H 5725 2850 50  0000 C CNN
-F 2 "" H 5650 3150 50  0000 C CNN
+F 2 "LEDs:LED_RGB_Getian_GT-P6PRGB4303" H 5650 3150 50  0001 C CNN
 F 3 "" H 5650 3150 50  0000 C CNN
 	1    5700 3200
@@
 F 0 "D4" H 5775 4350 50  0000 C CNN
 F 1 "LED_RABG" H 5725 3650 50  0000 C CNN
-F 2 "" H 5650 3950 50  0000 C CNN
+F 2 "LEDs:LED_RGB_Getian_GT-P6PRGB4303" H 5650 3950 50  0001 C CNN
 F 3 "" H 5650 3950 50  0000 C CNN
 	1    5700 4000
@@
 F 0 "D5" H 5775 5150 50  0000 C CNN
 F 1 "LED_RABG" H 5725 4450 50  0000 C CNN
-F 2 "" H 5650 4750 50  0000 C CNN
+F 2 "LEDs:LED_RGB_Getian_GT-P6PRGB4303" H 5650 4750 50  0001 C CNN
 F 3 "" H 5650 4750 50  0000 C CNN
 	1    5700 4800
@@
 F 0 "D6" H 5775 5950 50  0000 C CNN
 F 1 "LED_RABG" H 5725 5250 50  0000 C CNN
-F 2 "" H 5650 5550 50  0000 C CNN
+F 2 "LEDs:LED_RGB_Getian_GT-P6PRGB4303" H 5650 5550 50  0001 C CNN
 F 3 "" H 5650 5550 50  0000 C CNN
 	1    5700 5600
@@
 F 0 "D7" H 5775 6750 50  0000 C CNN
 F 1 "LED_RABG" H 5725 6050 50  0000 C CNN
-F 2 "" H 5650 6350 50  0000 C CNN
+F 2 "LEDs:LED_RGB_Getian_GT-P6PRGB4303" H 5650 6350 50  0001 C CNN
 F 3 "" H 5650 6350 50  0000 C CNN
 	1    5700 6400
@@
 F 0 "D8" H 5775 7550 50  0000 C CNN
 F 1 "LED_RABG" H 5725 6850 50  0000 C CNN
-F 2 "" H 5650 7150 50  0000 C CNN
+F 2 "LEDs:LED_RGB_Getian_GT-P6PRGB4303" H 5650 7150 50  0001 C CNN
 F 3 "" H 5650 7150 50  0000 C CNN
 	1    5700 7200
@@
 F 0 "R3" V 830 1200 50  0000 C CNN
 F 1 "R100" V 750 1200 50  0000 C CNN
-F 2 "" V 680 1200 30  0000 C CNN
+F 2 "Resistors_SMD:R_0402" V 680 1200 30  0001 C CNN
 F 3 "" H 750 1200 30  0000 C CNN
 	1    750  1200
@@
 F 0 "R4" V 2480 4100 50  0000 C CNN
 F 1 "R1K" V 2400 4100 50  0000 C CNN
-F 2 "" V 2330 4100 30  0000 C CNN
+F 2 "Resistors_SMD:R_0402" V 2330 4100 30  0001 C CNN
 F 3 "" H 2400 4100 30  0000 C CNN
 	1    2400 4100
@@
 F 0 "RP1" H 7150 2050 50  0000 C CNN
 F 1 "R_1K" H 7150 1550 50  0000 C CNN
-F 2 "" H 7150 1600 60  0000 C CNN
+F 2 "Resistors_SMD:R_0402" H 7150 1600 60  0001 C CNN
 F 3 "" H 7150 1600 60  0000 C CNN
 	1    7150 1600
@@
 F 0 "RP4" H 7700 2450 50  0000 C CNN
 F 1 "R_1K" H 7700 1950 50  0000 C CNN
-F 2 "" H 7700 2000 60  0000 C CNN
+F 2 "Resistors_SMD:R_0402" H 7700 2000 60  0001 C CNN
 F 3 "" H 7700 2000 60  0000 C CNN
 	1    7700 2000
@@
 F 0 "RP2" H 7150 4750 50  0000 C CNN
 F 1 "R_1K" H 7150 4250 50  0000 C CNN
-F 2 "" H 7150 4300 60  0000 C CNN
+F 2 "Resistors_SMD:R_0402" H 7150 4300 60  0001 C CNN
 F 3 "" H 7150 4300 60  0000 C CNN
 	1    7150 4300
@@
 F 0 "RP5" H 7700 5150 50  0000 C CNN
 F 1 "R_1K" H 7700 4650 50  0000 C CNN
-F 2 "" H 7700 4700 60  0000 C CNN
+F 2 "Resistors_SMD:R_0402" H 7700 4700 60  0001 C CNN
 F 3 "" H 7700 4700 60  0000 C CNN
 	1    7700 4700
@@
 F 0 "RP3" H 7150 7100 50  0000 C CNN
 F 1 "R_1K" H 7150 6600 50  0000 C CNN
-F 2 "" H 7150 6650 60  0000 C CNN
+F 2 "Resistors_SMD:R_0402" H 7150 6650 60  0001 C CNN
 F 3 "" H 7150 6650 60  0000 C CNN
 	1    7150 6650
@@
 F 0 "RP6" H 7700 7500 50  0000 C CNN
 F 1 "R_1K" H 7700 7000 50  0000 C CNN
-F 2 "" H 7700 7050 60  0000 C CNN
+F 2 "Resistors_SMD:R_0402" H 7700 7050 60  0001 C CNN
 F 3 "" H 7700 7050 60  0000 C CNN
 	1    7700 7050
@@
 F 0 "U1" H 4000 2850 50  0000 C CNN
 F 1 "74LS165" H 4000 2650 50  0000 C CNN
-F 2 "" H 3850 2900 50  0000 C CNN
+F 2 "Housings_SSOP:TSSOP-16_4.4x5mm_Pitch0.65mm" H 3850 2900 50  0001 C CNN
 F 3 "" H 3850 2900 50  0000 C CNN
 	1    3850 2900
@@
 F 0 "U2" H 9800 2300 70  0000 C CNN
 F 1 "74HC595" H 9650 1100 70  0000 C CNN
-F 2 "" H 9650 1700 60  0000 C CNN
+F 2 "Housings_SSOP:TSSOP-16_4.4x5mm_Pitch0.65mm" H 9650 1700 60  0001 C CNN
 F 3 "" H 9650 1700 60  0000 C CNN
 	1    9650 1700
@@
 F 0 "U3" H 9800 5000 70  0000 C CNN
 F 1 "74HC595" H 9650 3800 70  0000 C CNN
-F 2 "" H 9650 4400 60  0000 C CNN
+F 2 "Housings_SSOP:TSSOP-16_4.4x5mm_Pitch0.65mm" H 9650 4400 60  0001 C CNN
 F 3 "" H 9650 4400 60  0000 C CNN
 	1    9650 4400
@@
 F 0 "U4" H 9800 7350 70  0000 C CNN
 F 1 "74HC595" H 9650 6150 70  0000 C CNN
-F 2 "" H 9650 6750 60  0000 C CNN
+F 2 "Housings_SSOP:TSSOP-16_4.4x5mm_Pitch0.65mm" H 9650 6750 60  0001 C CNN
 F 3 "" H 9650 6750 60  0000 C CNN
 	1    9650 6750
