File: board/evm/circuit/battery.sch (KiCad schematic (older format))
At the start: 1 part

Commit message: add more schs
Parts:
- removed U?: nRF24LU1+, symbol nRF24LU1+
Changed lines of the file:
@@
 $Descr A4 11693 8268
 encoding utf-8
-Sheet 7 11
+Sheet 1 11
 Title ""
 Date ""
@@
 Comment4 ""
 $EndDescr
-$Comp
-L nRF24LU1+ U?
-U 1 1 5754763F
-P 3500 2850
-F 0 "U?" H 3500 2850 60  0000 C CNN
-F 1 "nRF24LU1+" H 3500 2750 60  0000 C CNN
-F 2 "" H 3500 2850 60  0000 C CNN
-F 3 "" H 3500 2850 60  0000 C CNN
-	1    3500 2850
-	1    0    0    -1
-$EndComp
 $EndSCHEMATC

Commit message: still working for sch
All done except for battery, which need more consideration on scheme of
QC2.0 (or QC3.0?), bidirectional charge.
Parts:
- added U?: BQ25895, symbol BQ25895
Changed lines of the file:
@@
 LIBS:contrib
 LIBS:valves
-LIBS:stm8
-LIBS:stm32
-LIBS:74xgxx
-LIBS:ac-dc
-LIBS:actel
 LIBS:Altera
-LIBS:analog_devices
-LIBS:battery_management
-LIBS:bbd
-LIBS:brooktre
-LIBS:cmos_ieee
-LIBS:dc-dc
-LIBS:diode
-LIBS:elec-unifil
-LIBS:ESD_Protection
-LIBS:ftdi
-LIBS:gennum
-LIBS:graphic
-LIBS:hc11
-LIBS:ir
-LIBS:Lattice
-LIBS:logo
-LIBS:maxim
-LIBS:microchip_dspic33dsc
-LIBS:microchip_pic10mcu
-LIBS:microchip_pic12mcu
-LIBS:microchip_pic16mcu
-LIBS:microchip_pic18mcu
-LIBS:microchip_pic32mcu
-LIBS:motor_drivers
-LIBS:msp430
-LIBS:nordicsemi
-LIBS:nxp_armmcu
-LIBS:onsemi
-LIBS:Oscillators
-LIBS:powerint
-LIBS:Power_Management
-LIBS:pspice
-LIBS:references
-LIBS:relays
-LIBS:rfcom
-LIBS:sensors
-LIBS:silabs
-LIBS:supertex
-LIBS:switches
-LIBS:transf
-LIBS:ttl_ieee
-LIBS:video
-LIBS:Worldsemi
-LIBS:Xicor
-LIBS:Zilog
 LIBS:my_kicad
 LIBS:oh-my-keyboard-cache
@@
 $Descr A4 11693 8268
 encoding utf-8
-Sheet 1 11
+Sheet 11 11
 Title ""
 Date ""
@@
 Comment4 ""
 $EndDescr
+$Comp
+L BQ25895 U?
+U 1 1 575B5A0D
+P 4950 3250
+F 0 "U?" H 4500 3650 60  0000 C CNN
+F 1 "BQ25895" H 4500 3300 60  0000 C CNN
+F 2 "" H 4950 3250 60  0000 C CNN
+F 3 "" H 4950 3250 60  0000 C CNN
+	1    4950 3250
+	1    0    0    -1
+$EndComp
 $EndSCHEMATC

Commit message: battery sch nearly done
Parts:
- added BT?: Li-Ion, symbol Battery
- added C? (x4): 10uF, symbol C_Small
- added C? (x2): 0.1uF, symbol C_Small
- added C?: 2.2uF, symbol C_Small
- added C?: 1uF, symbol C_Small
- added C? (x3): 22uF, symbol C_Small
- added C? (x2): 47nF, symbol C_Small
- added C? (x2): C_val, symbol C_Small
- added C?: 220nF, symbol C_Small
- added C?: 4.7nF, symbol C_Small
- added C?: 40uF, symbol C_Small
- added D?: LED, symbol LED
- added L?: 1.2uH/12A, symbol INDUCTOR
- added L?: 2.2uH, symbol INDUCTOR
- added P?: USB_A_flipable, symbol USB_A_flipable
- added P?: USB_OTG, symbol USB_OTG
- added R?: R255K, symbol R
- added R?: R360K, symbol R
- added R? (x2): R56K, symbol R
- added R?: R, symbol R
- added R? (x2): R2.2K, symbol R
- added R?: R260, symbol R
- added RP?: R_10K, symbol R_PACK4
- added U?: TPS61088, symbol TPS61088
- added U?: FP6601, symbol FP6601
Connections:
- net at U?.1 (VBUS): now also P?.1 (VCC)
- net at U?.10 (ILIM): now also R?.1
- net BAT+: now reaches U?.13 (BAT)
- net BAT+: now also U?.14 (BAT), BT?.1, C?.1, C?.1, C?.1, L?.2, U?.9 (VIN)
- net at U?.15 (SYS): now also U?.16 (SYS), C?.1, C?.1, L?.1
- net GND: now reaches U?.17 (PGND)
- net GND: now also U?.18 (PGND), BT?.2, C?.1, C?.1, C?.1, C?.1, C?.2, C?.2, C?.2, C?.2, C?.2, C?.2, C?.2, C?.2, C?.2, C?.2, C?.2, C?.2, P?.4 (GND), P?.5 (GND), P?.8 (GND), P?.9 (SHIELD), R?.2, R?.2, U?.2 (GND), U?.20 (AGND), U?.21 (PGND)
- net at U?.19 (SW): now also U?.20 (SW), C?.2, L?.2
- net at U?.2 (D+): now also P?.3 (D+)
- net at U?.21 (BTST): now also C?.1
- net at U?.22 (REGN): now also C?.2
- net at U?.23 (PMID): now also C?.2
- net at U?.3 (D-): now also P?.2 (D-)
- net at U?.4 (STAT): now also R?.1
- net BAT_SCL: now reaches U?.5 (SCL)
- net BAT_SCL: now also RP?.4 (P4)
- net BAT_SDA: now reaches U?.6 (SDA)
- net BAT_SDA: now also RP?.3 (P3)
- net BAT_INT: now reaches U?.7 (INT)
- net BAT_INT: now also RP?.2 (P2)
- net BAT_OTG: now reaches U?.8 (OTG)
- net BAT_nCE: now reaches U?.9 (nCE)
- new net: C?.1, U?.1 (VCC)
- new net: C?.1, U?.10 (SS)
- new net: R?.1, R?.1, U?.17 (FB)
- new net: C?.2, R?.1, U?.18 (COMP)
- new net: R?.1, U?.19 (ILIM)
- new net: R?.1, U?.3 (FSW)
- new net: C?.1, L?.1, R?.2, U?.4 (SW), U?.5 (SW), U?.6 (SW), U?.7 (SW)
- new net: C?.2, U?.8 (BOOT)
- new net: R?.2, U?.4 (VSEN2)
- new net: R?.2, U?.3 (VSEN1)
- new net: C?.2, R?.2
- new net: P?.3 (D+), P?.7 (D+), U?.1 (D+)
- new net: C?.1, R?.1, U?.5 (VDD)
- new net: P?.2 (D-), P?.6 (D-), U?.6 (D-)
- new net: D?.1 (K), R?.2
- new net +3V3: D?.2 (A), RP?.5 (R4), RP?.6 (R3), RP?.7 (R2), RP?.8 (R1)
- new net BatteryBoost_EN: U?.2 (EN)
- new net VBUS: C?.1, C?.1, C?.1, C?.1, P?.1 (VCC), P?.5 (VCC), R?.2, U?.14 (VOUT), U?.15 (VOUT), U?.16 (VOUT)
Other:
- note added: "<- FIXME"
- note added: "<- FIXME\nAdd short-circuit detection"
- moved on the sheet: U?

Commit message: refine battery circuit
Parts:
- removed C?: 40uF, symbol C_Small
- added C?: 40uF(DNI), symbol C_Small
- added D?: DNI, symbol D_Schottky_Small
- added R? (x2): R10K, symbol R
- added SW?: SW_PUSH, symbol SW_PUSH
Connections:
- net BAT_OTG is gone; now on net GND: U?.8 (OTG)
- net GND: now also U?.25 (PAD), C?.2, R?.1, SW?.2
- net at U?.11 (TS): now also R?.2, R?.2
- net at U?.12 (nQON): now also SW?.1
- net +BATT: now reaches C?.1, C?.1, L?.1, U?.15 (SYS), U?.16 (SYS)
- net at C?.2, L?.2, U?.19 (SW)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: now also D?.2 (A)
- net Device_D+: now reaches P?.3 (D+), U?.2 (D+)
- net REGN: now reaches C?.2, U?.22 (REGN)
- net REGN: now also R?.1
- net at U?.23 (PMID): now also C?.1, D?.1 (K)
- net BAT_DSEL: now reaches U?.24 (DSEL)
- net Device_D-: now reaches P?.2 (D-), U?.3 (D-)
Other:
- moved on the sheet: C?

Commit message: working on leak current detection
Parts:
- added C? (x4): 0.1uF, symbol C_Small
- added C? (x4): 20uF, symbol C_Small
- added D? (x2): D_SM340A, symbol D_Schottky
- added L? (x2): 3.3uH, symbol INDUCTOR
- added Q? (x3): Q_NMOS_DGS, symbol Q_NMOS_DGS
- added R? (x5): R10K, symbol R
- added R? (x2): R88K, symbol R
- added R? (x2): R12K, symbol R
- added R? (x2): R100K, symbol R
- added U? (x2): FP6291, symbol FP6291
- added U? (x2): NE5532, symbol LM358
Connections:
- net +3V3: now also C?.1, C?.1, D?.1 (K), R?.1
- net +BATT: now also C?.1, C?.1, C?.1, C?.1, L?.1, L?.1, U?.4 (EN), U?.4 (EN), U?.5 (VCC), U?.5 (VCC)
- net GND: now also C?.2, C?.2, C?.2, C?.2, C?.2, C?.2, C?.2, C?.2, R?.2, R?.2, R?.2, R?.2, U?.2 (GND), U?.2 (GND); no longer U?.8 (OTG)
- net VBUS: now also Q?.1 (D); no longer P?.1 (VCC), P?.5 (VCC)
- net +5V: now reaches C?.1, D?.1 (K), U?.23 (PMID)
- net Host_D+: now reaches P?.3 (D+), P?.7 (D+), U?.1 (D+)
- net Host_D-: now reaches P?.2 (D-), P?.6 (D-), U?.6 (D-)
- new net: Q?.1 (D), Q?.1 (D), Q?.3 (S), R?.1, R?.1
- new net: D?.2 (A), L?.2, U?.1 (LX) (x2)
- new net: R?.1, R?.2, U?.3 (FB) (x2)
- new net: R?.1, U?.6 (OC) (x2)
- new net: P?.1 (VCC), Q?.3 (S), R?.2
- new net: P?.5 (VCC), Q?.3 (S), R?.2
- new net +12V: C?.1, C?.1, D?.1 (K), R?.1, R?.1, R?.1, R?.1
- new net BAT_OTG_EN: U?.8 (OTG)
- new net ChargeOutputBypass1: Q?.2 (G), R?.2
- new net ChargeOutputBypass2: Q?.2 (G), R?.2
- new net ChargeOutputEN: Q?.2 (G), R?.2
Other:
- note added: "Boost to 12V"
- note added: "Boost to 3.3V"
- note added: "FIXME!"
- note added: "Provide QC2.0 Charge port for external devices"
- note added: "QC2.0 Charge to battery"
- moved on the sheet: BT?, C?, D?, L?, P?, R?, RP?, SW?, U?

Commit message: evm sch design finished
Parts:
- removed U? (x2): NE5532, symbol LM358
Connections:
- net HIGH_LOAD2: now reaches Q?.1 (D), Q?.1 (D), Q?.3 (S), R?.1, R?.1
- net HIGH_LOAD1: now reaches P?.5 (VCC), Q?.3 (S), R?.2
Other:
- note removed: "<- FIXME\nAdd short-circuit detection"
- moved on the sheet: BT?, C?, L?, P?, Q?, R?, U?

Commit message: bug fix
Changed lines of the file:
@@
 LIBS:Altera
 LIBS:my_kicad
+LIBS:Oscillators
 LIBS:oh-my-keyboard-cache
 EELAYER 25 0
@@
 $Descr A3 16535 11693
 encoding utf-8
-Sheet 11 12
+Sheet 10 12
 Title ""
 Date ""
@@
 	4900 7650 4350 7650
 Wire Wire Line
-	4350 7500 4350 7650
-Wire Wire Line
-	3150 7500 4350 7500
+	4350 7650 4350 7500
+Wire Wire Line
+	4350 7500 3150 7500
 Wire Wire Line
 	3150 7400 4500 7400
@@
 	4900 7950 4400 7950
 Wire Wire Line
-	4400 8350 4400 7950
-Wire Wire Line
-	3550 8350 4400 8350
+	4400 7950 4400 8350
+Wire Wire Line
+	4400 8350 3550 8350
 Text HLabel 3550 8350 0    60   Input ~ 0
 BAT_SCL
