File: board/evm/circuit/bluetooth.sch (KiCad schematic (older format))
At the start: 14 parts

Commit message: working on drc
Parts:
- gave numbers to parts that had none: 14
Connections:
- wire segments 63 -> 52
Changed lines of the file:
@@
 $EndDescr
 $Comp
-L DA14580-QFN40 U?
+L DA14580-QFN40 U8
 U 1 1 575491AD
 P 5400 3450
-F 0 "U?" H 5300 3500 60  0000 C CNN
+F 0 "U8" H 5300 3500 60  0000 C CNN
 F 1 "DA14580-QFN40" H 5350 3350 60  0000 C CNN
 F 2 "" H 5300 3500 60  0000 C CNN
@@
 SCL
 $Comp
-L +3V3 #PWR?
+L +3V3 #PWR068
 U 1 1 57594899
 P 1750 1000
-F 0 "#PWR?" H 1750 850 50  0001 C CNN
+F 0 "#PWR068" H 1750 850 50  0001 C CNN
 F 1 "+3V3" H 1750 1140 50  0000 C CNN
 F 2 "" H 1750 1000 50  0000 C CNN
@@
 	1750 1200 1750 1000
 $Comp
-L GND #PWR?
+L GND #PWR069
 U 1 1 575948B2
 P 1750 1500
-F 0 "#PWR?" H 1750 1250 50  0001 C CNN
+F 0 "#PWR069" H 1750 1250 50  0001 C CNN
 F 1 "GND" H 1750 1350 50  0000 C CNN
 F 2 "" H 1750 1500 50  0000 C CNN
@@
 	1750 1400 1750 1500
 $Comp
-L +3V3 #PWR?
+L +3V3 #PWR070
 U 1 1 575948CE
 P 4250 4450
-F 0 "#PWR?" H 4250 4300 50  0001 C CNN
+F 0 "#PWR070" H 4250 4300 50  0001 C CNN
 F 1 "+3V3" H 4250 4590 50  0000 C CNN
 F 2 "" H 4250 4450 50  0000 C CNN
@@
 	4250 4450 4250 4800
 Wire Wire Line
-	4250 4800 5150 4800
-Wire Wire Line
-	5150 4800 5250 4800
-Wire Wire Line
-	5150 4400 5150 4800
-Wire Wire Line
-	5150 4800 5150 4900
+	4250 4800 5250 4800
+Wire Wire Line
+	5150 4400 5150 4900
 Wire Wire Line
 	5250 4800 5250 4400
 Connection ~ 5150 4800
 $Comp
-L C_Small C?
+L C_Small C23
 U 1 1 57594902
 P 5150 5000
-F 0 "C?" H 5160 5070 50  0000 L CNN
+F 0 "C23" H 5160 5070 50  0000 L CNN
 F 1 "1uF" H 5160 4920 50  0000 L CNN
 F 2 "" H 5150 5000 50  0000 C CNN
@@
 $EndComp
 $Comp
-L GND #PWR?
+L GND #PWR071
 U 1 1 57594985
 P 5150 5250
-F 0 "#PWR?" H 5150 5000 50  0001 C CNN
+F 0 "#PWR071" H 5150 5000 50  0001 C CNN
 F 1 "GND" H 5150 5100 50  0000 C CNN
 F 2 "" H 5150 5250 50  0000 C CNN
@@
 $EndComp
 Wire Wire Line
-	5150 5100 5150 5200
-Wire Wire Line
-	5150 5200 5150 5250
+	5150 5100 5150 5250
 Wire Wire Line
 	5350 4400 5350 5200
@@
 Connection ~ 5150 5200
 $Comp
-L GND #PWR?
+L GND #PWR072
 U 1 1 575949DB
 P 6550 4200
-F 0 "#PWR?" H 6550 3950 50  0001 C CNN
+F 0 "#PWR072" H 6550 3950 50  0001 C CNN
 F 1 "GND" H 6550 4050 50  0000 C CNN
 F 2 "" H 6550 4200 50  0000 C CNN
@@
 	6400 4050 6550 4050
 Wire Wire Line
-	6550 3700 6550 4050
-Wire Wire Line
-	6550 4050 6550 4200
-$Comp
-L INDUCTOR_SMALL L?
+	6550 3700 6550 4200
+$Comp
+L INDUCTOR_SMALL L6
 U 1 1 57594A20
 P 6950 3900
-F 0 "L?" H 6950 4000 50  0000 C CNN
+F 0 "L6" H 6950 4000 50  0000 C CNN
 F 1 "2.2uH" H 6950 3850 50  0000 C CNN
 F 2 "" H 6950 3900 50  0000 C CNN
@@
 	6400 3900 6700 3900
 Wire Wire Line
-	7200 3900 7400 3900
-Wire Wire Line
-	7400 3900 7550 3900
+	7200 3900 7550 3900
 Wire Wire Line
 	7400 3900 7400 4700
@@
 VDCDC
 Wire Wire Line
-	5750 2000 5750 2200
-Wire Wire Line
-	5750 2200 5750 2500
+	5750 2000 5750 2500
 Text Label 5750 2400 1    60   ~ 0
 VDCDC
 $Comp
-L C_Small C?
+L C_Small C24
 U 1 1 57594AAC
 P 6000 2300
-F 0 "C?" H 6010 2370 50  0000 L CNN
+F 0 "C24" H 6010 2370 50  0000 L CNN
 F 1 "1uF" H 6010 2220 50  0000 L CNN
 F 2 "" H 6000 2300 50  0000 C CNN
@@
 Connection ~ 5750 2200
 $Comp
-L GND #PWR?
+L GND #PWR073
 U 1 1 57594B38
 P 6000 2450
-F 0 "#PWR?" H 6000 2200 50  0001 C CNN
+F 0 "#PWR073" H 6000 2200 50  0001 C CNN
 F 1 "GND" H 6000 2300 50  0000 C CNN
 F 2 "" H 6000 2450 50  0000 C CNN
@@
 Connection ~ 6550 4050
 $Comp
-L CRYSTAL_SMT Y?
+L CRYSTAL_SMT Y2
 U 1 1 57594EC4
 P 7200 2600
-F 0 "Y?" H 7200 2900 60  0000 C CNN
+F 0 "Y2" H 7200 2900 60  0000 C CNN
 F 1 "CRYSTAL_16M" H 7200 2800 60  0000 C CNN
 F 2 "" H 7200 2600 60  0000 C CNN
@@
 	6550 3100 6400 3100
 $Comp
-L GND #PWR?
+L GND #PWR074
 U 1 1 57594FC8
 P 7750 2750
-F 0 "#PWR?" H 7750 2500 50  0001 C CNN
+F 0 "#PWR074" H 7750 2500 50  0001 C CNN
 F 1 "GND" H 7750 2600 50  0000 C CNN
 F 2 "" H 7750 2750 50  0000 C CNN
@@
 	7750 2600 7750 2750
 $Comp
-L TagConnect J?
+L TagConnect J2
 U 1 1 57595027
 P 4150 1300
-F 0 "J?" H 3850 1150 60  0000 C CNN
+F 0 "J2" H 3850 1150 60  0000 C CNN
 F 1 "TagConnect" H 4350 1150 60  0000 C CNN
 F 2 "" H 4000 1350 60  0000 C CNN
@@
 $EndComp
 $Comp
-L +3V3 #PWR?
+L +3V3 #PWR075
 U 1 1 5759512A
 P 3400 1000
-F 0 "#PWR?" H 3400 850 50  0001 C CNN
+F 0 "#PWR075" H 3400 850 50  0001 C CNN
 F 1 "+3V3" H 3400 1140 50  0000 C CNN
 F 2 "" H 3400 1000 50  0000 C CNN
@@
 	3400 1150 3550 1150
 $Comp
-L GND #PWR?
+L GND #PWR076
 U 1 1 5759517F
 P 3400 1450
-F 0 "#PWR?" H 3400 1200 50  0001 C CNN
+F 0 "#PWR076" H 3400 1200 50  0001 C CNN
 F 1 "GND" H 3400 1300 50  0000 C CNN
 F 2 "" H 3400 1450 50  0000 C CNN
@@
 SWCLK
 $Comp
-L C_Small C?
+L C_Small C27
 U 1 1 575956A9
 P 7550 4000
-F 0 "C?" H 7560 4070 50  0000 L CNN
+F 0 "C27" H 7560 4070 50  0000 L CNN
 F 1 "1uF" H 7560 3920 50  0000 L CNN
 F 2 "" H 7550 4000 50  0000 C CNN
@@
 $EndComp
 $Comp
-L GND #PWR?
+L GND #PWR077
 U 1 1 57595724
 P 7550 4150
-F 0 "#PWR?" H 7550 3900 50  0001 C CNN
+F 0 "#PWR077" H 7550 3900 50  0001 C CNN
 F 1 "GND" H 7550 4000 50  0000 C CNN
 F 2 "" H 7550 4150 50  0000 C CNN
@@
 Connection ~ 7400 3900
 $Comp
-L L_Small L?
+L L_Small L4
 U 1 1 57595AEB
 P 6300 1650
-F 0 "L?" H 6330 1690 50  0000 L CNN
+F 0 "L4" H 6330 1690 50  0000 L CNN
 F 1 "3.3nH" H 6330 1610 50  0000 L CNN
 F 2 "" H 6300 1650 50  0000 C CNN
@@
 $EndComp
 $Comp
-L L_Small L?
+L L_Small L5
 U 1 1 57595B48
 P 6900 1550
-F 0 "L?" V 6850 1450 50  0000 L CNN
+F 0 "L5" V 6850 1450 50  0000 L CNN
 F 1 "4.3nH" V 7000 1600 50  0000 L CNN
 F 2 "" H 6900 1550 50  0000 C CNN
@@
 	5350 2500 5350 1550
 Wire Wire Line
-	5350 1550 6300 1550
-Wire Wire Line
-	6300 1550 6800 1550
+	5350 1550 6800 1550
 Connection ~ 6300 1550
 $Comp
-L C_Small C?
+L C_Small C25
 U 1 1 57595F02
 P 6650 1650
-F 0 "C?" H 6660 1720 50  0000 L CNN
+F 0 "C25" H 6660 1720 50  0000 L CNN
 F 1 "0.5pF" H 6660 1570 50  0000 L CNN
 F 2 "" H 6650 1650 50  0000 C CNN
@@
 	6300 1750 6300 1850
 Wire Wire Line
-	6300 1850 6650 1850
-Wire Wire Line
-	6650 1850 7250 1850
-Wire Wire Line
-	7250 1850 7550 1850
-Wire Wire Line
-	6650 1750 6650 1850
-Wire Wire Line
-	6650 1850 6650 1950
-$Comp
-L GND #PWR?
+	6300 1850 7550 1850
+Wire Wire Line
+	6650 1750 6650 1950
+$Comp
+L GND #PWR078
 U 1 1 57595FB6
 P 6650 1950
-F 0 "#PWR?" H 6650 1700 50  0001 C CNN
+F 0 "#PWR078" H 6650 1700 50  0001 C CNN
 F 1 "GND" H 6650 1800 50  0000 C CNN
 F 2 "" H 6650 1950 50  0000 C CNN
@@
 $EndComp
 $Comp
-L C_Small C?
+L C_Small C26
 U 1 1 57596029
 P 7250 1650
-F 0 "C?" H 7260 1720 50  0000 L CNN
+F 0 "C26" H 7260 1720 50  0000 L CNN
 F 1 "1.5pF" H 7260 1570 50  0000 L CNN
 F 2 "" H 7250 1650 50  0000 C CNN
@@
 $EndComp
 Wire Wire Line
-	7000 1550 7250 1550
-Wire Wire Line
-	7250 1550 7800 1550
+	7000 1550 7800 1550
 Wire Wire Line
 	7250 1850 7250 1750
 Connection ~ 6650 1850
 $Comp
-L ANTPCB E?
+L ANTPCB E2
 U 1 1 57596217
 P 7800 1500
-F 0 "E?" H 7700 1650 60  0000 C CNN
+F 0 "E2" H 7700 1650 60  0000 C CNN
 F 1 "ANTPCB" H 7800 1400 60  0000 C CNN
 F 2 "" H 7800 1500 60  0000 C CNN
@@
 Connection ~ 7250 1850
 $Comp
-L LED D?
+L LED D9
 U 1 1 57596385
 P 3300 3000
-F 0 "D?" H 3300 3100 50  0000 C CNN
+F 0 "D9" H 3300 3100 50  0000 C CNN
 F 1 "LED" H 3300 2900 50  0000 C CNN
 F 2 "" H 3300 3000 50  0000 C CNN
@@
 	3850 3000 4350 3000
 $Comp
-L R R?
+L R R7
 U 1 1 5759657F
 P 3700 3000
-F 0 "R?" V 3780 3000 50  0000 C CNN
+F 0 "R7" V 3780 3000 50  0000 C CNN
 F 1 "510" V 3700 3000 50  0000 C CNN
 F 2 "" V 3630 3000 50  0000 C CNN
@@
 	3550 3000 3500 3000
 $Comp
-L GND #PWR?
+L GND #PWR079
 U 1 1 5759667C
 P 3050 3150
-F 0 "#PWR?" H 3050 2900 50  0001 C CNN
+F 0 "#PWR079" H 3050 2900 50  0001 C CNN
 F 1 "GND" H 3050 3000 50  0000 C CNN
 F 2 "" H 3050 3150 50  0000 C CNN
