File: board/evm/circuit/bluetooth.sch (KiCad schematic (older format))
At the start: 14 parts, among them J2 TagConnect, U8 DA14580-QFN40, Y2 CRYSTAL_16M

Commit message: working on footprint
Parts:
- C23, C24, C27: footprint (none) -> Capacitors_SMD:C_0603
- C25, C26: footprint (none) -> Capacitors_SMD:C_0402
- D9: footprint (none) -> LEDs:LED_0805
- R7: footprint (none) -> Resistors_SMD:R_0402
- U8: footprint (none) -> Housings_DFN_QFN:QFN-40-1EP_5x5mm_Pitch0.4mm
Changed lines of the file:
@@
 F 0 "U8" H 5300 3500 60  0000 C CNN
 F 1 "DA14580-QFN40" H 5350 3350 60  0000 C CNN
-F 2 "" H 5300 3500 60  0000 C CNN
+F 2 "Housings_DFN_QFN:QFN-40-1EP_5x5mm_Pitch0.4mm" H 5300 3500 60  0001 C CNN
 F 3 "" H 5300 3500 60  0000 C CNN
 	1    5400 3450
@@
 F 0 "C23" H 5160 5070 50  0000 L CNN
 F 1 "1uF" H 5160 4920 50  0000 L CNN
-F 2 "" H 5150 5000 50  0000 C CNN
+F 2 "Capacitors_SMD:C_0603" H 5150 5000 50  0001 C CNN
 F 3 "" H 5150 5000 50  0000 C CNN
 	1    5150 5000
@@
 F 0 "L6" H 6950 4000 50  0000 C CNN
 F 1 "2.2uH" H 6950 3850 50  0000 C CNN
-F 2 "" H 6950 3900 50  0000 C CNN
+F 2 "" H 6950 3900 50  0001 C CNN
 F 3 "" H 6950 3900 50  0000 C CNN
 	1    6950 3900
@@
 F 0 "C24" H 6010 2370 50  0000 L CNN
 F 1 "1uF" H 6010 2220 50  0000 L CNN
-F 2 "" H 6000 2300 50  0000 C CNN
+F 2 "Capacitors_SMD:C_0603" H 6000 2300 50  0001 C CNN
 F 3 "" H 6000 2300 50  0000 C CNN
 	1    6000 2300
@@
 F 0 "Y2" H 7200 2900 60  0000 C CNN
 F 1 "CRYSTAL_16M" H 7200 2800 60  0000 C CNN
-F 2 "" H 7200 2600 60  0000 C CNN
+F 2 "" H 7200 2600 60  0001 C CNN
 F 3 "" H 7200 2600 60  0000 C CNN
 	1    7200 2600
@@
 F 0 "J2" H 3850 1150 60  0000 C CNN
 F 1 "TagConnect" H 4350 1150 60  0000 C CNN
-F 2 "" H 4000 1350 60  0000 C CNN
+F 2 "" H 4000 1350 60  0001 C CNN
 F 3 "" H 4000 1350 60  0000 C CNN
 	1    4150 1300
@@
 F 0 "C27" H 7560 4070 50  0000 L CNN
 F 1 "1uF" H 7560 3920 50  0000 L CNN
-F 2 "" H 7550 4000 50  0000 C CNN
+F 2 "Capacitors_SMD:C_0603" H 7550 4000 50  0001 C CNN
 F 3 "" H 7550 4000 50  0000 C CNN
 	1    7550 4000
@@
 F 0 "L4" H 6330 1690 50  0000 L CNN
 F 1 "3.3nH" H 6330 1610 50  0000 L CNN
-F 2 "" H 6300 1650 50  0000 C CNN
+F 2 "" H 6300 1650 50  0001 C CNN
 F 3 "" H 6300 1650 50  0000 C CNN
 	1    6300 1650
@@
 F 0 "L5" V 6850 1450 50  0000 L CNN
 F 1 "4.3nH" V 7000 1600 50  0000 L CNN
-F 2 "" H 6900 1550 50  0000 C CNN
+F 2 "" H 6900 1550 50  0001 C CNN
 F 3 "" H 6900 1550 50  0000 C CNN
 	1    6900 1550
@@
 F 0 "C25" H 6660 1720 50  0000 L CNN
 F 1 "0.5pF" H 6660 1570 50  0000 L CNN
-F 2 "" H 6650 1650 50  0000 C CNN
+F 2 "Capacitors_SMD:C_0402" H 6650 1650 50  0001 C CNN
 F 3 "" H 6650 1650 50  0000 C CNN
 	1    6650 1650
@@
 F 0 "C26" H 7260 1720 50  0000 L CNN
 F 1 "1.5pF" H 7260 1570 50  0000 L CNN
-F 2 "" H 7250 1650 50  0000 C CNN
+F 2 "Capacitors_SMD:C_0402" H 7250 1650 50  0001 C CNN
 F 3 "" H 7250 1650 50  0000 C CNN
 	1    7250 1650
@@
 F 0 "E2" H 7700 1650 60  0000 C CNN
 F 1 "ANTPCB" H 7800 1400 60  0000 C CNN
-F 2 "" H 7800 1500 60  0000 C CNN
+F 2 "" H 7800 1500 60  0001 C CNN
 F 3 "" H 7800 1500 60  0000 C CNN
 	1    7800 1500
@@
 F 0 "D9" H 3300 3100 50  0000 C CNN
 F 1 "LED" H 3300 2900 50  0000 C CNN
-F 2 "" H 3300 3000 50  0000 C CNN
+F 2 "LEDs:LED_0805" H 3300 3000 50  0001 C CNN
 F 3 "" H 3300 3000 50  0000 C CNN
 	1    3300 3000
@@
 F 0 "R7" V 3780 3000 50  0000 C CNN
 F 1 "510" V 3700 3000 50  0000 C CNN
-F 2 "" V 3630 3000 50  0000 C CNN
+F 2 "Resistors_SMD:R_0402" V 3630 3000 50  0001 C CNN
 F 3 "" H 3700 3000 50  0000 C CNN
 	1    3700 3000
