File: board/evm/circuit/mcu.sch (KiCad schematic (older format))
At the start: 28 parts

Commit message: change cpld to fpga due to limited resource
Connections:
- wire segments 118 -> 87
Changed lines of the file:
@@
 $EndComp
 Wire Wire Line
-	8000 2300 8000 2450
-Wire Wire Line
-	8000 2450 8000 2800
-Wire Wire Line
-	8000 2800 8000 3100
+	8000 2300 8000 3100
 Connection ~ 8000 3100
 Connection ~ 8100 3100
@@
 	8100 9000 8100 9150
 Wire Wire Line
-	8100 9000 8200 9000
-Wire Wire Line
-	8200 9000 8300 9000
-Wire Wire Line
-	8300 9000 8400 9000
-Wire Wire Line
-	8400 9000 8500 9000
+	8100 9000 8500 9000
 Connection ~ 8100 9000
 Connection ~ 8200 9000
@@
 $EndComp
 Wire Wire Line
-	8000 2450 8400 2450
-Wire Wire Line
-	8400 2450 8700 2450
-Wire Wire Line
-	8700 2450 9000 2450
-Wire Wire Line
-	9000 2450 9300 2450
-Wire Wire Line
-	9300 2450 9600 2450
-Wire Wire Line
-	9600 2450 9900 2450
-Wire Wire Line
-	9900 2450 10200 2450
-Wire Wire Line
-	10200 2450 10500 2450
+	8000 2450 10500 2450
 Connection ~ 8000 2450
 Connection ~ 8400 2450
@@
 Connection ~ 10200 2450
 Wire Wire Line
-	8400 2650 8700 2650
-Wire Wire Line
-	8700 2650 9000 2650
-Wire Wire Line
-	9000 2650 9300 2650
-Wire Wire Line
-	9300 2650 9600 2650
-Wire Wire Line
-	9600 2650 9900 2650
-Wire Wire Line
-	9900 2650 10200 2650
-Wire Wire Line
-	10200 2650 10500 2650
+	8400 2650 10500 2650
 Connection ~ 8700 2650
 Connection ~ 9000 2650
@@
 	1550 3200 1550 3150
 Wire Wire Line
-	1550 3500 1550 3600
-Wire Wire Line
-	1550 3600 1550 3750
+	1550 3500 1550 3750
 Wire Wire Line
 	2150 3600 3800 3600
@@
 $EndComp
 Wire Wire Line
-	2750 4100 3700 4100
-Wire Wire Line
-	3700 4100 3800 4100
+	2750 4100 3800 4100
 $Comp
 L GND #PWR?
@@
 $EndComp
 Wire Wire Line
-	8000 3100 8100 3100
-Wire Wire Line
-	8100 3100 8200 3100
-Wire Wire Line
-	8200 3100 8300 3100
-Wire Wire Line
-	8300 3100 8400 3100
-Wire Wire Line
-	8400 3100 8500 3100
+	8000 3100 8500 3100
 $Comp
 L L_Small L?
@@
 	8600 3100 8600 3000
 Wire Wire Line
-	8000 2800 8600 2800
-Wire Wire Line
-	8600 2800 8800 2800
+	8000 2800 8800 2800
 Connection ~ 8000 2800
 $Comp
@@
 	3650 4300 3800 4300
 Wire Wire Line
-	3350 4500 3350 4600
-Wire Wire Line
-	3350 4600 3350 4650
+	3350 4500 3350 4650
 Wire Wire Line
 	3650 4500 3650 4600
@@
 Wire Wire Line
 	12800 4700 13850 4700
-Wire Wire Line
-	13850 4700 13850 4700
 Wire Wire Line
 	12800 4800 13850 4800
@@
 	14800 3050 14700 3050
 Wire Wire Line
-	14800 2750 14800 2850
-Wire Wire Line
-	14800 2850 14800 3050
-Wire Wire Line
-	14800 3050 14800 3150
+	14800 2750 14800 3150
 $Comp
 L GND #PWR?
@@
 Text HLabel 12800 5100 2    60   Input ~ 0
 SPI3_NSS
-Text HLabel 12800 6200 2    60   Input ~ 0
+Text HLabel 12800 6500 2    60   Input ~ 0
 SPI2_NSS
 Text HLabel 12800 6300 2    60   Input ~ 0
@@
 	12800 3900 12800 3900
 Wire Wire Line
-	12800 4500 12800 4500
-Wire Wire Line
-	12800 4600 12800 4600
+	12800 4500 15050 4500
+Wire Wire Line
+	12800 4600 15150 4600
 Wire Wire Line
 	12800 4900 13150 4900
@@
 Wire Wire Line
 	13300 8400 12800 8400
-NoConn ~ 12800 6500
 NoConn ~ 12800 6100
 NoConn ~ 3800 5300
@@
 	3750 3800 3800 3800
 Wire Wire Line
-	12800 4500 15050 4500
-Wire Wire Line
-	12800 4600 15150 4600
-Wire Wire Line
 	15150 4600 15150 4500
 $Comp
@@
 Text Label 13450 4600 0    60   ~ 0
 USART_TTL_RX
+NoConn ~ 12800 6200
 $EndSCHEMATC

Commit message: working on drc
Parts:
- gave numbers to parts that had none: 28
