File: board/evm/circuit/mcu.sch (KiCad schematic (older format))
At the start: 28 parts, among them J5 TagConnect, P6 CONN_01X03, SW10 SW_PUSH, U24 STM32F405VGTx, U25 W25Q32, Y4 CRYSTAL_8M

Commit message: working on footprint
Parts:
- C79, C80, C81: footprint (none) -> Capacitors_SMD:C_0603
- C82, C83, C85, C86, C87, C88, C89, C90: footprint (none) -> Capacitors_SMD:C_0402
- C84: footprint (none) -> Capacitors_SMD:C_0805
- D19: footprint (none) -> LEDs:LED_0805
- L14: footprint (none) -> Resistors_SMD:R_0805
- R56, R57, R58, R59, R60, R61, R62, R63: footprint (none) -> Resistors_SMD:R_0402
- SW10: footprint (none) -> Buttons_Switches_SMD:SW_SPST_B3U-1000P
- U24: footprint LQFP100 -> Housings_QFP:LQFP-100_14x14mm_Pitch0.5mm
- Y4: value CRYSTAL_8M -> CRYSTAL_16M
Changed lines of the file:
@@
 F 0 "U24" H 4000 8925 50  0000 L BNN
 F 1 "STM32F405VGTx" H 12600 8925 50  0000 R BNN
-F 2 "LQFP100" H 12600 8875 50  0000 R TNN
+F 2 "Housings_QFP:LQFP-100_14x14mm_Pitch0.5mm" H 12600 8875 50  0000 R TNN
 F 3 "" H 8300 6100 50  0000 C CNN
 	1    8300 6100
@@
 F 0 "C87" H 9610 2620 50  0000 L CNN
 F 1 "C_104" H 9610 2470 50  0000 L CNN
-F 2 "" H 9600 2550 50  0000 C CNN
+F 2 "Capacitors_SMD:C_0402" H 9600 2550 50  0001 C CNN
 F 3 "" H 9600 2550 50  0000 C CNN
 	1    9600 2550
@@
 F 0 "C88" H 9910 2620 50  0000 L CNN
 F 1 "C_104" H 9910 2470 50  0000 L CNN
-F 2 "" H 9900 2550 50  0000 C CNN
+F 2 "Capacitors_SMD:C_0402" H 9900 2550 50  0001 C CNN
 F 3 "" H 9900 2550 50  0000 C CNN
 	1    9900 2550
@@
 F 0 "C89" H 10210 2620 50  0000 L CNN
 F 1 "C_104" H 10210 2470 50  0000 L CNN
-F 2 "" H 10200 2550 50  0000 C CNN
+F 2 "Capacitors_SMD:C_0402" H 10200 2550 50  0001 C CNN
 F 3 "" H 10200 2550 50  0000 C CNN
 	1    10200 2550
@@
 F 0 "C90" H 10510 2620 50  0000 L CNN
 F 1 "C_104" H 10510 2470 50  0000 L CNN
-F 2 "" H 10500 2550 50  0000 C CNN
+F 2 "Capacitors_SMD:C_0402" H 10500 2550 50  0001 C CNN
 F 3 "" H 10500 2550 50  0000 C CNN
 	1    10500 2550
@@
 F 0 "C82" H 8410 2620 50  0000 L CNN
 F 1 "C_104" H 8410 2470 50  0000 L CNN
-F 2 "" H 8400 2550 50  0000 C CNN
+F 2 "Capacitors_SMD:C_0402" H 8400 2550 50  0001 C CNN
 F 3 "" H 8400 2550 50  0000 C CNN
 	1    8400 2550
@@
 F 0 "C83" H 8710 2620 50  0000 L CNN
 F 1 "C_104" H 8710 2470 50  0000 L CNN
-F 2 "" H 8700 2550 50  0000 C CNN
+F 2 "Capacitors_SMD:C_0402" H 8700 2550 50  0001 C CNN
 F 3 "" H 8700 2550 50  0000 C CNN
 	1    8700 2550
@@
 F 0 "C85" H 9010 2620 50  0000 L CNN
 F 1 "C_104" H 9010 2470 50  0000 L CNN
-F 2 "" H 9000 2550 50  0000 C CNN
+F 2 "Capacitors_SMD:C_0402" H 9000 2550 50  0001 C CNN
 F 3 "" H 9000 2550 50  0000 C CNN
 	1    9000 2550
@@
 F 0 "C86" H 9310 2620 50  0000 L CNN
 F 1 "C_104" H 9310 2470 50  0000 L CNN
-F 2 "" H 9300 2550 50  0000 C CNN
+F 2 "Capacitors_SMD:C_0402" H 9300 2550 50  0001 C CNN
 F 3 "" H 9300 2550 50  0000 C CNN
 	1    9300 2550
@@
 F 0 "R59" V 13630 6700 50  0000 C CNN
 F 1 "R22" V 13550 6700 50  0000 C CNN
-F 2 "" V 13480 6700 50  0000 C CNN
+F 2 "Resistors_SMD:R_0402" V 13480 6700 50  0001 C CNN
 F 3 "" H 13550 6700 50  0000 C CNN
 	1    13550 6700
@@
 F 0 "R60" V 13630 6900 50  0000 C CNN
 F 1 "R22" V 13550 6900 50  0000 C CNN
-F 2 "" V 13480 6900 50  0000 C CNN
+F 2 "Resistors_SMD:R_0402" V 13480 6900 50  0001 C CNN
 F 3 "" H 13550 6900 50  0000 C CNN
 	1    13550 6900
@@
 F 0 "SW10" H 2000 3710 50  0000 C CNN
 F 1 "SW_PUSH" H 1850 3520 50  0000 C CNN
-F 2 "" H 1850 3600 50  0000 C CNN
+F 2 "Buttons_Switches_SMD:SW_SPST_B3U-1000P" H 1850 3600 50  0001 C CNN
 F 3 "" H 1850 3600 50  0000 C CNN
 	1    1850 3600
@@
 F 0 "R56" V 1630 3350 50  0000 C CNN
 F 1 "R1K" V 1550 3350 50  0000 C CNN
-F 2 "" V 1480 3350 50  0000 C CNN
+F 2 "Resistors_SMD:R_0402" V 1480 3350 50  0001 C CNN
 F 3 "" H 1550 3350 50  0000 C CNN
 	1    1550 3350
@@
 F 0 "C79" H 1560 3920 50  0000 L CNN
 F 1 "C_105" H 1560 3770 50  0000 L CNN
-F 2 "" H 1550 3850 50  0000 C CNN
+F 2 "Capacitors_SMD:C_0603" H 1550 3850 50  0001 C CNN
 F 3 "" H 1550 3850 50  0000 C CNN
 	1    1550 3850
@@
 F 0 "L14" H 8630 2940 50  0000 L CNN
 F 1 "Bead" H 8630 2860 50  0000 L CNN
-F 2 "" H 8600 2900 50  0000 C CNN
+F 2 "Resistors_SMD:R_0805" H 8600 2900 50  0001 C CNN
 F 3 "" H 8600 2900 50  0000 C CNN
 	1    8600 2900
@@
 F 0 "C84" H 8810 2970 50  0000 L CNN
 F 1 "C_106" H 8810 2820 50  0000 L CNN
-F 2 "" H 8800 2900 50  0000 C CNN
+F 2 "Capacitors_SMD:C_0805" H 8800 2900 50  0001 C CNN
 F 3 "" H 8800 2900 50  0000 C CNN
 	1    8800 2900
@@
 F 0 "C80" H 3360 4470 50  0000 L CNN
 F 1 "C_225" H 3360 4320 50  0000 L CNN
-F 2 "" H 3350 4400 50  0000 C CNN
+F 2 "Capacitors_SMD:C_0603" H 3350 4400 50  0001 C CNN
 F 3 "" H 3350 4400 50  0000 C CNN
 	1    3350 4400
@@
 F 0 "C81" H 3660 4470 50  0000 L CNN
 F 1 "C_225" H 3660 4320 50  0000 L CNN
-F 2 "" H 3650 4400 50  0000 C CNN
+F 2 "Capacitors_SMD:C_0603" H 3650 4400 50  0001 C CNN
 F 3 "" H 3650 4400 50  0000 C CNN
 	1    3650 4400
@@
 F 0 "R62" V 14080 4700 50  0000 C CNN
 F 1 "R22" V 14000 4700 50  0000 C CNN
-F 2 "" V 13930 4700 50  0000 C CNN
+F 2 "Resistors_SMD:R_0402" V 13930 4700 50  0001 C CNN
 F 3 "" H 14000 4700 50  0000 C CNN
 	1    14000 4700
@@
 F 0 "R63" V 14080 4850 50  0000 C CNN
 F 1 "R22" V 14000 4850 50  0000 C CNN
-F 2 "" V 13930 4850 50  0000 C CNN
+F 2 "Resistors_SMD:R_0402" V 13930 4850 50  0001 C CNN
 F 3 "" H 14000 4850 50  0000 C CNN
 	1    14000 4850
@@
 P 2500 5100
 F 0 "Y4" V 2500 5400 60  0000 C CNN
-F 1 "CRYSTAL_8M" V 2950 5200 60  0000 C CNN
-F 2 "" H 2500 5100 60  0000 C CNN
+F 1 "CRYSTAL_16M" V 2950 5200 60  0000 C CNN
+F 2 "" H 2500 5100 60  0001 C CNN
 F 3 "" H 2500 5100 60  0000 C CNN
 	1    2500 5100
@@
 F 0 "U25" H 13950 3400 60  0000 C CNN
 F 1 "W25Q32" H 13950 2950 60  0000 C CNN
-F 2 "" H 13950 3200 60  0000 C CNN
+F 2 "" H 13950 3200 60  0001 C CNN
 F 3 "" H 13950 3200 60  0000 C CNN
 	1    13950 3200
@@
 F 0 "R58" V 13230 5500 50  0000 C CNN
 F 1 "R10K" V 13150 5500 50  0000 C CNN
-F 2 "" V 13080 5500 50  0000 C CNN
+F 2 "Resistors_SMD:R_0402" V 13080 5500 50  0001 C CNN
 F 3 "" H 13150 5500 50  0000 C CNN
 	1    13150 5500
@@
 F 0 "J5" H 16450 5400 60  0000 C CNN
 F 1 "TagConnect" H 16950 5400 60  0000 C CNN
-F 2 "" H 16600 5600 60  0000 C CNN
+F 2 "" H 16600 5600 60  0001 C CNN
 F 3 "" H 16600 5600 60  0000 C CNN
 	1    16750 5550
@@
 F 0 "D19" H 13500 8500 50  0000 C CNN
 F 1 "LED" H 13500 8300 50  0000 C CNN
-F 2 "" H 13500 8400 50  0000 C CNN
+F 2 "LEDs:LED_0805" H 13500 8400 50  0001 C CNN
 F 3 "" H 13500 8400 50  0000 C CNN
 	1    13500 8400
@@
 F 0 "R61" V 13980 8400 50  0000 C CNN
 F 1 "R1K" V 13900 8400 50  0000 C CNN
-F 2 "" V 13830 8400 50  0000 C CNN
+F 2 "Resistors_SMD:R_0402" V 13830 8400 50  0001 C CNN
 F 3 "" H 13900 8400 50  0000 C CNN
 	1    13900 8400
@@
 F 0 "R57" V 3680 3800 50  0000 C CNN
 F 1 "R10K" V 3600 3800 50  0000 C CNN
-F 2 "" V 3530 3800 50  0000 C CNN
+F 2 "Resistors_SMD:R_0402" V 3530 3800 50  0001 C CNN
 F 3 "" H 3600 3800 50  0000 C CNN
 	1    3600 3800
@@
 F 0 "P6" H 15150 4500 50  0000 C CNN
 F 1 "CONN_01X03" V 15250 4300 50  0000 C CNN
-F 2 "" H 15150 4300 50  0000 C CNN
+F 2 "" H 15150 4300 50  0001 C CNN
 F 3 "" H 15150 4300 50  0000 C CNN
 	1    15150 4300

Commit message: still working on footprint
Parts:
- U25: footprint (none) -> Housings_SOIC:SOIC-8_3.9x4.9mm_Pitch1.27mm
Changed lines of the file:
@@
 LIBS:contrib
 LIBS:valves
+LIBS:stm8
+LIBS:stm32
+LIBS:74xgxx
+LIBS:ac-dc
+LIBS:actel
 LIBS:Altera
+LIBS:analog_devices
+LIBS:battery_management
+LIBS:bbd
+LIBS:brooktre
+LIBS:cmos_ieee
+LIBS:dc-dc
+LIBS:diode
+LIBS:elec-unifil
+LIBS:ESD_Protection
+LIBS:ftdi
+LIBS:gennum
+LIBS:graphic
+LIBS:hc11
+LIBS:ir
+LIBS:Lattice
+LIBS:logo
+LIBS:maxim
+LIBS:microchip_dspic33dsc
+LIBS:microchip_pic10mcu
+LIBS:microchip_pic12mcu
+LIBS:microchip_pic16mcu
+LIBS:microchip_pic18mcu
+LIBS:microchip_pic32mcu
+LIBS:motor_drivers
+LIBS:msp430
+LIBS:nordicsemi
+LIBS:nxp_armmcu
+LIBS:onsemi
+LIBS:Oscillators
+LIBS:powerint
+LIBS:Power_Management
+LIBS:pspice
+LIBS:references
+LIBS:relays
+LIBS:rfcom
+LIBS:sensors
+LIBS:silabs
+LIBS:supertex
+LIBS:switches
+LIBS:transf
+LIBS:ttl_ieee
+LIBS:video
+LIBS:Worldsemi
+LIBS:Xicor
+LIBS:Zilog
 LIBS:my_kicad
-LIBS:Oscillators
 LIBS:oh-my-keyboard-cache
 EELAYER 25 0
@@
 F 0 "U25" H 13950 3400 60  0000 C CNN
 F 1 "W25Q32" H 13950 2950 60  0000 C CNN
-F 2 "" H 13950 3200 60  0001 C CNN
+F 2 "Housings_SOIC:SOIC-8_3.9x4.9mm_Pitch1.27mm" H 13950 3200 60  0001 C CNN
 F 3 "" H 13950 3200 60  0000 C CNN
 	1    13950 3200
