File: board/evm/circuit/trackpoint.sch (KiCad schematic (older format))
At the start: 1 part

Commit message: working on drc
Parts:
- gave numbers to parts that had none: 1
Changed lines of the file:
@@
 $EndDescr
 $Comp
-L CONN_01X10 P?
+L CONN_01X10 P3
 U 1 1 5759DE16
 P 4150 2050
-F 0 "P?" H 4150 2600 50  0000 C CNN
+F 0 "P3" H 4150 2600 50  0000 C CNN
 F 1 "CONN_01X10" V 4250 2050 50  0000 C CNN
 F 2 "" H 4150 2050 50  0000 C CNN
