File: board/evm/circuit/trackpoint.sch (KiCad schematic (older format))
At the start: 0 parts

Commit message: still working for sch
All done except for battery, which need more consideration on scheme of
QC2.0 (or QC3.0?), bidirectional charge.
Parts:
- added P?: CONN_01X10, symbol CONN_01X10
Connections:
- new net BUTTON0: P?.3 (P3)
- new net BUTTON1: P?.2 (P2)
- new net BUTTON2: P?.1 (P1)
- new net EX.CKL: P?.7 (P7)
- new net EX.DATA: P?.9 (P9)
- new net GND: P?.6 (P6)
- new net RST: P?.10 (P10)
- new net TP_CLK: P?.4 (P4)
- new net TP_DATA: P?.8 (P8)
- new net VCC: P?.5 (P5)
Changed lines of the file:
@@
 LIBS:contrib
 LIBS:valves
-LIBS:stm8
-LIBS:stm32
-LIBS:74xgxx
-LIBS:ac-dc
-LIBS:actel
 LIBS:Altera
-LIBS:analog_devices
-LIBS:battery_management
-LIBS:bbd
-LIBS:brooktre
-LIBS:cmos_ieee
-LIBS:dc-dc
-LIBS:diode
-LIBS:elec-unifil
-LIBS:ESD_Protection
-LIBS:ftdi
-LIBS:gennum
-LIBS:graphic
-LIBS:hc11
-LIBS:ir
-LIBS:Lattice
-LIBS:logo
-LIBS:maxim
-LIBS:microchip_dspic33dsc
-LIBS:microchip_pic10mcu
-LIBS:microchip_pic12mcu
-LIBS:microchip_pic16mcu
-LIBS:microchip_pic18mcu
-LIBS:microchip_pic32mcu
-LIBS:motor_drivers
-LIBS:msp430
-LIBS:nordicsemi
-LIBS:nxp_armmcu
-LIBS:onsemi
-LIBS:Oscillators
-LIBS:powerint
-LIBS:Power_Management
-LIBS:pspice
-LIBS:references
-LIBS:relays
-LIBS:rfcom
-LIBS:sensors
-LIBS:silabs
-LIBS:supertex
-LIBS:switches
-LIBS:transf
-LIBS:ttl_ieee
-LIBS:video
-LIBS:Worldsemi
-LIBS:Xicor
-LIBS:Zilog
 LIBS:my_kicad
 LIBS:oh-my-keyboard-cache
@@
 $Descr A4 11693 8268
 encoding utf-8
-Sheet 1 11
+Sheet 9 11
 Title ""
 Date ""
@@
 Comment4 ""
 $EndDescr
+$Comp
+L CONN_01X10 P?
+U 1 1 5759DE16
+P 4150 2050
+F 0 "P?" H 4150 2600 50  0000 C CNN
+F 1 "CONN_01X10" V 4250 2050 50  0000 C CNN
+F 2 "" H 4150 2050 50  0000 C CNN
+F 3 "" H 4150 2050 50  0000 C CNN
+	1    4150 2050
+	1    0    0    -1
+$EndComp
+Text HLabel 3950 1600 0    60   Input ~ 0
+BUTTON2
+Text HLabel 3950 1700 0    60   Input ~ 0
+BUTTON1
+Text HLabel 3950 1800 0    60   Input ~ 0
+BUTTON0
+Text HLabel 3950 1900 0    60   Input ~ 0
+TP_CLK
+Text HLabel 3950 2000 0    60   Input ~ 0
+VCC
+Text HLabel 3950 2100 0    60   Input ~ 0
+GND
+Text HLabel 3950 2200 0    60   Input ~ 0
+EX.CKL
+Text HLabel 3950 2300 0    60   Input ~ 0
+TP_DATA
+Text HLabel 3950 2400 0    60   Input ~ 0
+EX.DATA
+Text HLabel 3950 2500 0    60   Input ~ 0
+RST
 $EndSCHEMATC

Commit message: working on qc3
Parts:
- gave numbers to parts that had none: 1
Changed lines of the file:
@@
 LIBS:contrib
 LIBS:valves
+LIBS:stm8
+LIBS:stm32
+LIBS:74xgxx
+LIBS:ac-dc
+LIBS:actel
 LIBS:Altera
-LIBS:my_kicad
+LIBS:analog_devices
+LIBS:battery_management
+LIBS:bbd
+LIBS:brooktre
+LIBS:cmos_ieee
+LIBS:dc-dc
+LIBS:diode
+LIBS:elec-unifil
+LIBS:ESD_Protection
+LIBS:ftdi
+LIBS:gennum
+LIBS:graphic
+LIBS:hc11
+LIBS:ir
+LIBS:Lattice
+LIBS:logo
+LIBS:maxim
+LIBS:microchip_dspic33dsc
+LIBS:microchip_pic10mcu
+LIBS:microchip_pic12mcu
+LIBS:microchip_pic16mcu
+LIBS:microchip_pic18mcu
+LIBS:microchip_pic32mcu
+LIBS:motor_drivers
+LIBS:msp430
+LIBS:nordicsemi
+LIBS:nxp_armmcu
+LIBS:onsemi
 LIBS:Oscillators
+LIBS:powerint
+LIBS:Power_Management
+LIBS:pspice
+LIBS:references
+LIBS:relays
+LIBS:rfcom
+LIBS:sensors
+LIBS:silabs
+LIBS:supertex
+LIBS:switches
+LIBS:transf
+LIBS:ttl_ieee
+LIBS:video
+LIBS:Worldsemi
+LIBS:Xicor
+LIBS:Zilog
 LIBS:oh-my-keyboard-cache
 EELAYER 25 0
@@
 $EndDescr
 $Comp
-L CONN_01X10 P?
+L CONN_01X10 P3
 U 1 1 5759DE16
 P 4150 2050
-F 0 "P?" H 4150 2600 50  0000 C CNN
+F 0 "P3" H 4150 2600 50  0000 C CNN
 F 1 "CONN_01X10" V 4250 2050 50  0000 C CNN
 F 2 "" H 4150 2050 50  0000 C CNN
