File: board/evm/circuit/CurrentSense.sch (KiCad schematic (older format))
At the start: 55 parts

Commit message: working on qc3
Parts:
- gave numbers to parts that had none: 53
Connections:
- net DETECT_I2C_SDA: now also U21.6 (COLLECTOR); no longer U21.7 (COLLECTOR)
- net HIGH_LOAD2: now also U19.6 (-); no longer U19.2 (-)
- net I2C_SDA: now also U21.3 (CATHODE); no longer U21.2 (CATHODE)
- net SIGNAL2: now also U19.7; no longer U19.1
- net at R43.2, R47.1: now also U19.5 (+); no longer U19.3 (+)
- net at R51.1: now also U21.4 (ANODE); no longer U21.1 (ANODE)
