File: board/evm/circuit/CurrentSense.sch (KiCad schematic (older format))
At the start: 46 parts

Commit message: minor updates
- add lots of test points
- export usart1
- bug fix
Parts:
- added W? (x9): TP, symbol TEST_1P
Other:
- note added: "Isolated GND"
- moved on the sheet: C?, R?, U?, U?A

Commit message: working on drc
Parts:
- gave numbers to parts that had none: 53
Connections:
- net DETECT_I2C_SDA: now also U22.6 (COLLECTOR); no longer U22.7 (COLLECTOR)
- net HIGH_LOAD2: now also U20.6 (-); no longer U20.2 (-)
- net I2C_SDA: now also U22.3 (CATHODE); no longer U22.2 (CATHODE)
- net SIGNAL2: now also U20.7; no longer U20.1
- net at R45.2, R49.1: now also U20.5 (+); no longer U20.3 (+)
- net at R53.1: now also U22.4 (ANODE); no longer U22.1 (ANODE)

Commit message: working on footprint
Parts:
- C65, C66, C67, C69, C72, C73, C74, C75, C76, C77, C78: footprint (none) -> Capacitors_SMD:C_0402
- C68, C70, C71: footprint (none) -> Capacitors_SMD:C_0805
- D15, D16, D17: footprint (none) -> Diodes_SMD:SMA_Standard
- D18: footprint (none) -> LEDs:LED_0805
- R39, R40, R41, R42, R43, R44, R45, R46, R47, R48, R49, R50, R51, R52, R53, R54, R55: footprint (none) -> Resistors_SMD:R_0402
- U18: footprint DIP-4 -> Housings_DIP:DIP-4_W7.62mm
- U21: footprint (none) -> TO_SOT_Packages_SMD:SOT-223
- U23: footprint (none) -> Housings_DFN_QFN:UQFN-20-1EP_3x3mm_Pitch0.4mm
- W54, W55, W56, W57, W58, W59, W60, W61, W62: footprint (none) -> Connect:PINTST

Commit message: still working on footprint
Parts:
- U17: footprint (none) -> Housings_SOIC:SOIC-8-1EP_3.9x4.9mm_Pitch1.27mm
- U20, U22: footprint (none) -> Housings_SOIC:SOIC-8_3.9x4.9mm_Pitch1.27mm
Changed lines of the file:
@@
 LIBS:contrib
 LIBS:valves
+LIBS:stm8
+LIBS:stm32
+LIBS:74xgxx
+LIBS:ac-dc
+LIBS:actel
 LIBS:Altera
+LIBS:analog_devices
+LIBS:battery_management
+LIBS:bbd
+LIBS:brooktre
+LIBS:cmos_ieee
+LIBS:dc-dc
+LIBS:diode
+LIBS:elec-unifil
+LIBS:ESD_Protection
+LIBS:ftdi
+LIBS:gennum
+LIBS:graphic
+LIBS:hc11
+LIBS:ir
+LIBS:Lattice
+LIBS:logo
+LIBS:maxim
+LIBS:microchip_dspic33dsc
+LIBS:microchip_pic10mcu
+LIBS:microchip_pic12mcu
+LIBS:microchip_pic16mcu
+LIBS:microchip_pic18mcu
+LIBS:microchip_pic32mcu
+LIBS:motor_drivers
+LIBS:msp430
+LIBS:nordicsemi
+LIBS:nxp_armmcu
+LIBS:onsemi
+LIBS:Oscillators
+LIBS:powerint
+LIBS:Power_Management
+LIBS:pspice
+LIBS:references
+LIBS:relays
+LIBS:rfcom
+LIBS:sensors
+LIBS:silabs
+LIBS:supertex
+LIBS:switches
+LIBS:transf
+LIBS:ttl_ieee
+LIBS:video
+LIBS:Worldsemi
+LIBS:Xicor
+LIBS:Zilog
 LIBS:my_kicad
-LIBS:Oscillators
 LIBS:oh-my-keyboard-cache
 EELAYER 25 0
@@
 F 0 "U17" H 2450 2500 60  0000 C CNN
 F 1 "MP2467" H 2400 1900 60  0000 C CNN
-F 2 "" H 2650 1900 60  0001 C CNN
+F 2 "Housings_SOIC:SOIC-8-1EP_3.9x4.9mm_Pitch1.27mm" H 2650 1900 60  0001 C CNN
 F 3 "" H 2650 1900 60  0000 C CNN
 	1    2400 2200
@@
 F 0 "U20" H 7950 1900 50  0000 L CNN
 F 1 "NE5532" H 7950 1450 50  0000 L CNN
-F 2 "" H 8000 1700 50  0001 C CNN
+F 2 "Housings_SOIC:SOIC-8_3.9x4.9mm_Pitch1.27mm" H 8000 1700 50  0001 C CNN
 F 3 "" H 8000 1700 50  0000 C CNN
 	1    8000 1700
@@
 F 0 "U20" H 7950 3950 50  0000 L CNN
 F 1 "NE5532" H 7950 3500 50  0000 L CNN
-F 2 "" H 8000 3750 50  0001 C CNN
+F 2 "Housings_SOIC:SOIC-8_3.9x4.9mm_Pitch1.27mm" H 8000 3750 50  0001 C CNN
 F 3 "" H 8000 3750 50  0000 C CNN
 	2    8000 3750
@@
 F 0 "U22" H 12370 5450 50  0000 C CNN
 F 1 "HCPL2630" H 12520 5150 50  0000 C CNN
-F 2 "" H 11900 5300 50  0001 C CNN
+F 2 "Housings_SOIC:SOIC-8_3.9x4.9mm_Pitch1.27mm" H 11900 5300 50  0001 C CNN
 F 3 "" H 11900 5300 50  0000 C CNN
 	1    11900 5300
@@
 F 0 "U22" H 12370 6900 50  0000 C CNN
 F 1 "HCPL2630" H 12520 6600 50  0000 C CNN
-F 2 "" H 11900 6750 50  0001 C CNN
+F 2 "Housings_SOIC:SOIC-8_3.9x4.9mm_Pitch1.27mm" H 11900 6750 50  0001 C CNN
 F 3 "" H 11900 6750 50  0000 C CNN
 	2    11900 6750
