File: board/evm/circuit/nrf24l01.sch (KiCad schematic (older format))
At the start: 16 parts

Commit message: working on qc3
Parts:
- Y1: renamed from Y?; value CRYSTAL _16M -> CRYSTAL_16M
- gave numbers to parts that had none: 15
