File: board/evm/circuit/nrf24l01.sch (KiCad schematic (older format))
At the start: 16 parts, among them U7 nRF24L01, Y1 CRYSTAL _16M

Commit message: working on footprint
Parts:
- C14, C15: footprint (none) -> Capacitors_SMD:C_0603
- C16, C17, C18, C19, C20, C21, C22: footprint (none) -> Capacitors_SMD:C_0402
- R6: footprint (none) -> Resistors_SMD:R_0402
- U7: footprint (none) -> Housings_DFN_QFN:QFN-20-1EP_4x4mm_Pitch0.5mm
Changed lines of the file:
@@
 F 0 "U7" H 3050 2250 60  0000 C CNN
 F 1 "nRF24L01" H 3050 2400 60  0000 C CNN
-F 2 "" H 3450 1700 60  0000 C CNN
+F 2 "Housings_DFN_QFN:QFN-20-1EP_4x4mm_Pitch0.5mm" H 3450 1700 60  0001 C CNN
 F 3 "" H 3450 1700 60  0000 C CNN
 	1    3050 2250
@@
 F 0 "R6" V 3330 1250 50  0000 C CNN
 F 1 "R22K" V 3250 1250 50  0000 C CNN
-F 2 "" V 3180 1250 50  0000 C CNN
+F 2 "Resistors_SMD:R_0402" V 3180 1250 50  0001 C CNN
 F 3 "" H 3250 1250 50  0000 C CNN
 	1    3250 1250
@@
 F 0 "C16" H 2960 1570 50  0000 L CNN
 F 1 "33nF" H 2960 1420 50  0000 L CNN
-F 2 "" H 2950 1500 50  0000 C CNN
+F 2 "Capacitors_SMD:C_0402" H 2950 1500 50  0001 C CNN
 F 3 "" H 2950 1500 50  0000 C CNN
 	1    2950 1500
@@
 F 0 "C17" H 2960 3370 50  0000 L CNN
 F 1 "10nF" H 2960 3220 50  0000 L CNN
-F 2 "" H 2950 3300 50  0000 C CNN
+F 2 "Capacitors_SMD:C_0402" H 2950 3300 50  0001 C CNN
 F 3 "" H 2950 3300 50  0000 C CNN
 	1    2950 3300
@@
 F 0 "C18" H 4210 2120 50  0000 L CNN
 F 1 "10nF" H 4210 1970 50  0000 L CNN
-F 2 "" H 4200 2050 50  0000 C CNN
+F 2 "Capacitors_SMD:C_0402" H 4200 2050 50  0001 C CNN
 F 3 "" H 4200 2050 50  0000 C CNN
 	1    4200 2050
@@
 F 0 "C15" H 2560 1570 50  0000 L CNN
 F 1 "10nF" H 2560 1420 50  0000 L CNN
-F 2 "" H 2550 1500 50  0000 C CNN
+F 2 "Capacitors_SMD:C_0603" H 2550 1500 50  0001 C CNN
 F 3 "" H 2550 1500 50  0000 C CNN
 	1    2550 1500
@@
 F 0 "C14" H 2310 1570 50  0000 L CNN
 F 1 "10nF" H 2310 1420 50  0000 L CNN
-F 2 "" H 2300 1500 50  0000 C CNN
+F 2 "Capacitors_SMD:C_0603" H 2300 1500 50  0001 C CNN
 F 3 "" H 2300 1500 50  0000 C CNN
 	1    2300 1500
@@
 F 0 "Y1" H 3550 3600 60  0000 C CNN
 F 1 "CRYSTAL_16M" H 3550 3500 60  0000 C CNN
-F 2 "" H 3550 3300 60  0000 C CNN
+F 2 "" H 3550 3300 60  0001 C CNN
 F 3 "" H 3550 3300 60  0000 C CNN
 	1    3550 3300
@@
 F 0 "C19" H 4310 2620 50  0000 L CNN
 F 1 "2.2nF" H 4100 2450 50  0000 L CNN
-F 2 "" H 4300 2550 50  0000 C CNN
+F 2 "Capacitors_SMD:C_0402" H 4300 2550 50  0001 C CNN
 F 3 "" H 4300 2550 50  0000 C CNN
 	1    4300 2550
@@
 F 0 "C20" H 4610 2620 50  0000 L CNN
 F 1 "4.7pF" H 4610 2470 50  0000 L CNN
-F 2 "" H 4600 2550 50  0000 C CNN
+F 2 "Capacitors_SMD:C_0402" H 4600 2550 50  0001 C CNN
 F 3 "" H 4600 2550 50  0000 C CNN
 	1    4600 2550
@@
 F 0 "L1" H 4880 1990 50  0000 L CNN
 F 1 "8.2nH" H 4880 1910 50  0000 L CNN
-F 2 "" H 4850 1950 50  0000 C CNN
+F 2 "" H 4850 1950 50  0001 C CNN
 F 3 "" H 4850 1950 50  0000 C CNN
 	1    4850 1950
@@
 F 0 "L3" V 5050 2200 50  0000 L CNN
 F 1 "2.7nH" V 5200 2150 50  0000 L CNN
-F 2 "" H 5100 2200 50  0000 C CNN
+F 2 "" H 5100 2200 50  0001 C CNN
 F 3 "" H 5100 2200 50  0000 C CNN
 	1    5100 2200
@@
 F 0 "L2" V 5050 1550 50  0000 L CNN
 F 1 "3.9nH" V 5200 1500 50  0000 L CNN
-F 2 "" H 5100 1550 50  0000 C CNN
+F 2 "" H 5100 1550 50  0001 C CNN
 F 3 "" H 5100 1550 50  0000 C CNN
 	1    5100 1550
@@
 F 0 "C22" H 5500 1950 50  0000 L CNN
 F 1 "1.0pF" H 5650 1750 50  0000 L CNN
-F 2 "" H 5600 1850 50  0000 C CNN
+F 2 "Capacitors_SMD:C_0402" H 5600 1850 50  0001 C CNN
 F 3 "" H 5600 1850 50  0000 C CNN
 	1    5600 1850
@@
 F 0 "C21" V 5300 1650 50  0000 L CNN
 F 1 "1.5pF" V 5500 1450 50  0000 L CNN
-F 2 "" H 5400 1550 50  0000 C CNN
+F 2 "Capacitors_SMD:C_0402" H 5400 1550 50  0001 C CNN
 F 3 "" H 5400 1550 50  0000 C CNN
 	1    5400 1550
@@
 F 0 "E1" H 5850 1650 60  0000 C CNN
 F 1 "ANTPCB" H 5950 1400 60  0000 C CNN
-F 2 "" H 5950 1500 60  0000 C CNN
+F 2 "" H 5950 1500 60  0001 C CNN
 F 3 "" H 5950 1500 60  0000 C CNN
 	1    5950 1500

Commit message: still working on footprint
Parts:
- Y1: value CRYSTAL _16M -> CRYSTAL_16M
Changed lines of the file:
@@
 LIBS:contrib
 LIBS:valves
+LIBS:stm8
+LIBS:stm32
+LIBS:74xgxx
+LIBS:ac-dc
+LIBS:actel
 LIBS:Altera
+LIBS:analog_devices
+LIBS:battery_management
+LIBS:bbd
+LIBS:brooktre
+LIBS:cmos_ieee
+LIBS:dc-dc
+LIBS:diode
+LIBS:elec-unifil
+LIBS:ESD_Protection
+LIBS:ftdi
+LIBS:gennum
+LIBS:graphic
+LIBS:hc11
+LIBS:ir
+LIBS:Lattice
+LIBS:logo
+LIBS:maxim
+LIBS:microchip_dspic33dsc
+LIBS:microchip_pic10mcu
+LIBS:microchip_pic12mcu
+LIBS:microchip_pic16mcu
+LIBS:microchip_pic18mcu
+LIBS:microchip_pic32mcu
+LIBS:motor_drivers
+LIBS:msp430
+LIBS:nordicsemi
+LIBS:nxp_armmcu
+LIBS:onsemi
+LIBS:Oscillators
+LIBS:powerint
+LIBS:Power_Management
+LIBS:pspice
+LIBS:references
+LIBS:relays
+LIBS:rfcom
+LIBS:sensors
+LIBS:silabs
+LIBS:supertex
+LIBS:switches
+LIBS:transf
+LIBS:ttl_ieee
+LIBS:video
+LIBS:Worldsemi
+LIBS:Xicor
+LIBS:Zilog
 LIBS:my_kicad
-LIBS:Oscillators
 LIBS:oh-my-keyboard-cache
 EELAYER 25 0
@@
 P 3550 3300
 F 0 "Y1" H 3550 3600 60  0000 C CNN
-F 1 "CRYSTAL_16M" H 3550 3500 60  0000 C CNN
+F 1 "CRYSTAL_16M" H 3550 3500 60  0000 C CNN
 F 2 "" H 3550 3300 60  0001 C CNN
 F 3 "" H 3550 3300 60  0000 C CNN
