File: board/evm/circuit/touch.sch (KiCad schematic (older format))
At the start: 17 parts

Commit message: working on drc
Parts:
- gave numbers to parts that had none: 17
Changed lines of the file:
@@
 $EndDescr
 $Comp
-L MPR121QR2 U?
+L MPR121QR2 U10
 U 1 1 57549F10
 P 3850 2950
-F 0 "U?" H 3800 2900 60  0000 C CNN
+F 0 "U10" H 3800 2900 60  0000 C CNN
 F 1 "MPR121QR2" H 3850 3050 60  0000 C CNN
 F 2 "" H 4000 2700 60  0000 C CNN
@@
 TOUCH_SDA
 $Comp
-L GND #PWR?
+L GND #PWR097
 U 1 1 575A98BD
 P 2950 3950
-F 0 "#PWR?" H 2950 3700 50  0001 C CNN
+F 0 "#PWR097" H 2950 3700 50  0001 C CNN
 F 1 "GND" H 2950 3800 50  0000 C CNN
 F 2 "" H 2950 3950 50  0000 C CNN
@@
 	2950 3050 3150 3050
 $Comp
-L C_Small C?
+L C_Small C36
 U 1 1 575A98EA
 P 3050 3350
-F 0 "C?" H 3060 3420 50  0000 L CNN
+F 0 "C36" H 3060 3420 50  0000 L CNN
 F 1 "0.1uF" H 3060 3270 50  0000 L CNN
 F 2 "" H 3050 3350 50  0000 C CNN
@@
 Connection ~ 3050 3600
 $Comp
-L R R?
+L R R15
 U 1 1 575A9CC6
 P 3600 3800
-F 0 "R?" V 3680 3800 50  0000 C CNN
+F 0 "R15" V 3680 3800 50  0000 C CNN
 F 1 "R75K 1%" V 3500 3800 50  0000 C CNN
 F 2 "" V 3530 3800 50  0000 C CNN
@@
 	3750 3600 3750 3800
 $Comp
-L +3V3 #PWR?
+L +3V3 #PWR098
 U 1 1 575A9D6D
 P 2450 1850
-F 0 "#PWR?" H 2450 1700 50  0001 C CNN
+F 0 "#PWR098" H 2450 1700 50  0001 C CNN
 F 1 "+3V3" H 2450 1990 50  0000 C CNN
 F 2 "" H 2450 1850 50  0000 C CNN
@@
 $EndComp
 $Comp
-L R_PACK4 RP?
+L R_PACK4 RP7
 U 1 1 575A9D87
 P 2600 2400
-F 0 "RP?" H 2600 2850 50  0000 C CNN
+F 0 "RP7" H 2600 2850 50  0000 C CNN
 F 1 "R_10K" H 2600 2350 50  0000 C CNN
 F 2 "" H 2600 2400 50  0000 C CNN
@@
 Connection ~ 2450 2000
 $Comp
-L C_Small C?
+L C_Small C37
 U 1 1 575A9EDB
 P 3250 2150
-F 0 "C?" H 3260 2220 50  0000 L CNN
+F 0 "C37" H 3260 2220 50  0000 L CNN
 F 1 "0.1uF" H 3260 2070 50  0000 L CNN
 F 2 "" H 3250 2150 50  0000 C CNN
@@
 Connection ~ 3250 2000
 $Comp
-L GND #PWR?
+L GND #PWR099
 U 1 1 575A9F4D
 P 3250 2300
-F 0 "#PWR?" H 3250 2050 50  0001 C CNN
+F 0 "#PWR099" H 3250 2050 50  0001 C CNN
 F 1 "GND" H 3250 2150 50  0000 C CNN
 F 2 "" H 3250 2300 50  0000 C CNN
@@
 	3250 2300 3250 2250
 $Comp
-L TEST_1P W?
+L TEST_1P W37
 U 1 1 575A9FA1
 P 4650 1600
-F 0 "W?" H 4650 1870 50  0000 C CNN
+F 0 "W37" H 4650 1870 50  0000 C CNN
 F 1 "TEST_1P" H 4650 1800 50  0000 C CNN
 F 2 "" H 4850 1600 50  0000 C CNN
@@
 $EndComp
 $Comp
-L TEST_1P W?
+L TEST_1P W38
 U 1 1 575AA01E
 P 5000 1600
-F 0 "W?" H 5000 1870 50  0000 C CNN
+F 0 "W38" H 5000 1870 50  0000 C CNN
 F 1 "TEST_1P" H 5000 1800 50  0000 C CNN
 F 2 "" H 5200 1600 50  0000 C CNN
@@
 $EndComp
 $Comp
-L TEST_1P W?
+L TEST_1P W39
 U 1 1 575AA400
 P 5350 1600
-F 0 "W?" H 5350 1870 50  0000 C CNN
+F 0 "W39" H 5350 1870 50  0000 C CNN
 F 1 "TEST_1P" H 5350 1800 50  0000 C CNN
 F 2 "" H 5550 1600 50  0000 C CNN
@@
 $EndComp
 $Comp
-L TEST_1P W?
+L TEST_1P W40
 U 1 1 575AA436
 P 5700 1600
-F 0 "W?" H 5700 1870 50  0000 C CNN
+F 0 "W40" H 5700 1870 50  0000 C CNN
 F 1 "TEST_1P" H 5700 1800 50  0000 C CNN
 F 2 "" H 5900 1600 50  0000 C CNN
@@
 $EndComp
 $Comp
-L TEST_1P W?
+L TEST_1P W41
 U 1 1 575AA46B
 P 6050 1600
-F 0 "W?" H 6050 1870 50  0000 C CNN
+F 0 "W41" H 6050 1870 50  0000 C CNN
 F 1 "TEST_1P" H 6050 1800 50  0000 C CNN
 F 2 "" H 6250 1600 50  0000 C CNN
@@
 $EndComp
 $Comp
-L TEST_1P W?
+L TEST_1P W42
 U 1 1 575AA4A4
 P 6400 1600
-F 0 "W?" H 6400 1870 50  0000 C CNN
+F 0 "W42" H 6400 1870 50  0000 C CNN
 F 1 "TEST_1P" H 6400 1800 50  0000 C CNN
 F 2 "" H 6600 1600 50  0000 C CNN
@@
 $EndComp
 $Comp
-L TEST_1P W?
+L TEST_1P W43
 U 1 1 575AA4CB
 P 6750 1600
-F 0 "W?" H 6750 1870 50  0000 C CNN
+F 0 "W43" H 6750 1870 50  0000 C CNN
 F 1 "TEST_1P" H 6750 1800 50  0000 C CNN
 F 2 "" H 6950 1600 50  0000 C CNN
@@
 $EndComp
 $Comp
-L TEST_1P W?
+L TEST_1P W44
 U 1 1 575AA4F6
 P 7100 1600
-F 0 "W?" H 7100 1870 50  0000 C CNN
+F 0 "W44" H 7100 1870 50  0000 C CNN
 F 1 "TEST_1P" H 7100 1800 50  0000 C CNN
 F 2 "" H 7300 1600 50  0000 C CNN
@@
 $EndComp
 $Comp
-L TEST_1P W?
+L TEST_1P W45
 U 1 1 575AA523
 P 7450 1600
-F 0 "W?" H 7450 1870 50  0000 C CNN
+F 0 "W45" H 7450 1870 50  0000 C CNN
 F 1 "TEST_1P" H 7450 1800 50  0000 C CNN
 F 2 "" H 7650 1600 50  0000 C CNN
@@
 $EndComp
 $Comp
-L TEST_1P W?
+L TEST_1P W46
 U 1 1 575AA554
 P 7800 1600
-F 0 "W?" H 7800 1870 50  0000 C CNN
+F 0 "W46" H 7800 1870 50  0000 C CNN
 F 1 "TEST_1P" H 7800 1800 50  0000 C CNN
 F 2 "" H 8000 1600 50  0000 C CNN
@@
 $EndComp
 $Comp
-L TEST_1P W?
+L TEST_1P W47
 U 1 1 575AA58F
 P 8150 1600
-F 0 "W?" H 8150 1870 50  0000 C CNN
+F 0 "W47" H 8150 1870 50  0000 C CNN
 F 1 "TEST_1P" H 8150 1800 50  0000 C CNN
 F 2 "" H 8350 1600 50  0000 C CNN
@@
 $EndComp
 $Comp
-L TEST_1P W?
+L TEST_1P W48
 U 1 1 575AA5CA
 P 8550 1600
-F 0 "W?" H 8550 1870 50  0000 C CNN
+F 0 "W48" H 8550 1870 50  0000 C CNN
 F 1 "TEST_1P" H 8550 1800 50  0000 C CNN
 F 2 "" H 8750 1600 50  0000 C CNN
@@
 GND
 $Comp
-L +3V3 #PWR?
+L +3V3 #PWR0100
 U 1 1 575ACD48
 P 1400 1000
-F 0 "#PWR?" H 1400 850 50  0001 C CNN
+F 0 "#PWR0100" H 1400 850 50  0001 C CNN
 F 1 "+3V3" H 1400 1140 50  0000 C CNN
 F 2 "" H 1400 1000 50  0000 C CNN
@@
 	1400 1150 1400 1000
 $Comp
-L GND #PWR?
+L GND #PWR0101
 U 1 1 575ACDE0
 P 1400 1450
-F 0 "#PWR?" H 1400 1200 50  0001 C CNN
+F 0 "#PWR0101" H 1400 1200 50  0001 C CNN
 F 1 "GND" H 1400 1300 50  0000 C CNN
 F 2 "" H 1400 1450 50  0000 C CNN

Commit message: working on footprint
Parts:
- C36, C37: footprint (none) -> Capacitors_SMD:C_0402
- R15, RP7: footprint (none) -> Resistors_SMD:R_0402
- U10: footprint (none) -> Housings_DFN_QFN:UQFN-20-1EP_3x3mm_Pitch0.4mm
- W37, W38, W39, W40, W41, W42, W43, W44, W45, W46, W47, W48: footprint (none) -> Connect:PINTST
Changed lines of the file:
@@
 F 0 "U10" H 3800 2900 60  0000 C CNN
 F 1 "MPR121QR2" H 3850 3050 60  0000 C CNN
-F 2 "" H 4000 2700 60  0000 C CNN
+F 2 "Housings_DFN_QFN:UQFN-20-1EP_3x3mm_Pitch0.4mm" H 4000 2700 60  0001 C CNN
 F 3 "" H 4000 2700 60  0000 C CNN
 	1    3850 2950
@@
 F 0 "C36" H 3060 3420 50  0000 L CNN
 F 1 "0.1uF" H 3060 3270 50  0000 L CNN
-F 2 "" H 3050 3350 50  0000 C CNN
+F 2 "Capacitors_SMD:C_0402" H 3050 3350 50  0001 C CNN
 F 3 "" H 3050 3350 50  0000 C CNN
 	1    3050 3350
@@
 F 0 "R15" V 3680 3800 50  0000 C CNN
 F 1 "R75K 1%" V 3500 3800 50  0000 C CNN
-F 2 "" V 3530 3800 50  0000 C CNN
+F 2 "Resistors_SMD:R_0402" V 3530 3800 50  0001 C CNN
 F 3 "" H 3600 3800 50  0000 C CNN
 	1    3600 3800
@@
 F 0 "RP7" H 2600 2850 50  0000 C CNN
 F 1 "R_10K" H 2600 2350 50  0000 C CNN
-F 2 "" H 2600 2400 50  0000 C CNN
+F 2 "Resistors_SMD:R_0402" H 2600 2400 50  0001 C CNN
 F 3 "" H 2600 2400 50  0000 C CNN
 	1    2600 2400
@@
 F 0 "C37" H 3260 2220 50  0000 L CNN
 F 1 "0.1uF" H 3260 2070 50  0000 L CNN
-F 2 "" H 3250 2150 50  0000 C CNN
+F 2 "Capacitors_SMD:C_0402" H 3250 2150 50  0001 C CNN
 F 3 "" H 3250 2150 50  0000 C CNN
 	1    3250 2150
@@
 F 0 "W37" H 4650 1870 50  0000 C CNN
 F 1 "TEST_1P" H 4650 1800 50  0000 C CNN
-F 2 "" H 4850 1600 50  0000 C CNN
+F 2 "Connect:PINTST" H 4850 1600 50  0001 C CNN
 F 3 "" H 4850 1600 50  0000 C CNN
 	1    4650 1600
@@
 F 0 "W38" H 5000 1870 50  0000 C CNN
 F 1 "TEST_1P" H 5000 1800 50  0000 C CNN
-F 2 "" H 5200 1600 50  0000 C CNN
+F 2 "Connect:PINTST" H 5200 1600 50  0001 C CNN
 F 3 "" H 5200 1600 50  0000 C CNN
 	1    5000 1600
@@
 F 0 "W39" H 5350 1870 50  0000 C CNN
 F 1 "TEST_1P" H 5350 1800 50  0000 C CNN
-F 2 "" H 5550 1600 50  0000 C CNN
+F 2 "Connect:PINTST" H 5550 1600 50  0001 C CNN
 F 3 "" H 5550 1600 50  0000 C CNN
 	1    5350 1600
@@
 F 0 "W40" H 5700 1870 50  0000 C CNN
 F 1 "TEST_1P" H 5700 1800 50  0000 C CNN
-F 2 "" H 5900 1600 50  0000 C CNN
+F 2 "Connect:PINTST" H 5900 1600 50  0001 C CNN
 F 3 "" H 5900 1600 50  0000 C CNN
 	1    5700 1600
@@
 F 0 "W41" H 6050 1870 50  0000 C CNN
 F 1 "TEST_1P" H 6050 1800 50  0000 C CNN
-F 2 "" H 6250 1600 50  0000 C CNN
+F 2 "Connect:PINTST" H 6250 1600 50  0001 C CNN
 F 3 "" H 6250 1600 50  0000 C CNN
 	1    6050 1600
@@
 F 0 "W42" H 6400 1870 50  0000 C CNN
 F 1 "TEST_1P" H 6400 1800 50  0000 C CNN
-F 2 "" H 6600 1600 50  0000 C CNN
+F 2 "Connect:PINTST" H 6600 1600 50  0001 C CNN
 F 3 "" H 6600 1600 50  0000 C CNN
 	1    6400 1600
@@
 F 0 "W43" H 6750 1870 50  0000 C CNN
 F 1 "TEST_1P" H 6750 1800 50  0000 C CNN
-F 2 "" H 6950 1600 50  0000 C CNN
+F 2 "Connect:PINTST" H 6950 1600 50  0001 C CNN
 F 3 "" H 6950 1600 50  0000 C CNN
 	1    6750 1600
@@
 F 0 "W44" H 7100 1870 50  0000 C CNN
 F 1 "TEST_1P" H 7100 1800 50  0000 C CNN
-F 2 "" H 7300 1600 50  0000 C CNN
+F 2 "Connect:PINTST" H 7300 1600 50  0001 C CNN
 F 3 "" H 7300 1600 50  0000 C CNN
 	1    7100 1600
@@
 F 0 "W45" H 7450 1870 50  0000 C CNN
 F 1 "TEST_1P" H 7450 1800 50  0000 C CNN
-F 2 "" H 7650 1600 50  0000 C CNN
+F 2 "Connect:PINTST" H 7650 1600 50  0001 C CNN
 F 3 "" H 7650 1600 50  0000 C CNN
 	1    7450 1600
@@
 F 0 "W46" H 7800 1870 50  0000 C CNN
 F 1 "TEST_1P" H 7800 1800 50  0000 C CNN
-F 2 "" H 8000 1600 50  0000 C CNN
+F 2 "Connect:PINTST" H 8000 1600 50  0001 C CNN
 F 3 "" H 8000 1600 50  0000 C CNN
 	1    7800 1600
@@
 F 0 "W47" H 8150 1870 50  0000 C CNN
 F 1 "TEST_1P" H 8150 1800 50  0000 C CNN
-F 2 "" H 8350 1600 50  0000 C CNN
+F 2 "Connect:PINTST" H 8350 1600 50  0001 C CNN
 F 3 "" H 8350 1600 50  0000 C CNN
 	1    8150 1600
@@
 F 0 "W48" H 8550 1870 50  0000 C CNN
 F 1 "TEST_1P" H 8550 1800 50  0000 C CNN
-F 2 "" H 8750 1600 50  0000 C CNN
+F 2 "Connect:PINTST" H 8750 1600 50  0001 C CNN
 F 3 "" H 8750 1600 50  0000 C CNN
 	1    8550 1600
