File: board/evm/circuit/OLED.sch (KiCad schematic (older format))
At the start: 1 part

Commit message: working on drc
Parts:
- gave numbers to parts that had none: 1
Changed lines of the file:
@@
 $EndDescr
 $Comp
-L OLED-12864 U?
+L OLED-12864 U11
 U 1 1 5759530E
 P 3900 2550
-F 0 "U?" H 3800 2950 60  0000 C CNN
+F 0 "U11" H 3800 2950 60  0000 C CNN
 F 1 "OLED-12864" H 3800 2750 60  0000 C CNN
 F 2 "" H 2850 1850 60  0000 C CNN
@@
 GND
 $Comp
-L GND #PWR?
+L GND #PWR0102
 U 1 1 575AD12D
 P 5350 3600
-F 0 "#PWR?" H 5350 3350 50  0001 C CNN
+F 0 "#PWR0102" H 5350 3350 50  0001 C CNN
 F 1 "GND" H 5350 3450 50  0000 C CNN
 F 2 "" H 5350 3600 50  0000 C CNN
@@
 $EndComp
 $Comp
-L +3V3 #PWR?
+L +3V3 #PWR0103
 U 1 1 575AD192
 P 4450 3600
-F 0 "#PWR?" H 4450 3450 50  0001 C CNN
+F 0 "#PWR0103" H 4450 3450 50  0001 C CNN
 F 1 "+3V3" H 4450 3740 50  0000 C CNN
 F 2 "" H 4450 3600 50  0000 C CNN
@@
 $EndComp
 $Comp
-L +3V3 #PWR?
+L +3V3 #PWR0104
 U 1 1 575AD1C6
 P 1650 1200
-F 0 "#PWR?" H 1650 1050 50  0001 C CNN
+F 0 "#PWR0104" H 1650 1050 50  0001 C CNN
 F 1 "+3V3" H 1650 1340 50  0000 C CNN
 F 2 "" H 1650 1200 50  0000 C CNN
@@
 	1650 1350 1650 1200
 $Comp
-L GND #PWR?
+L GND #PWR0105
 U 1 1 575AD218
 P 1650 1700
-F 0 "#PWR?" H 1650 1450 50  0001 C CNN
+F 0 "#PWR0105" H 1650 1450 50  0001 C CNN
 F 1 "GND" H 1650 1550 50  0000 C CNN
 F 2 "" H 1650 1700 50  0000 C CNN
@@
 	1650 1550 1650 1700
 $Comp
-L +12V #PWR?
+L +12V #PWR0106
 U 1 1 575AE2B2
 P 2550 3800
-F 0 "#PWR?" H 2550 3650 50  0001 C CNN
+F 0 "#PWR0106" H 2550 3650 50  0001 C CNN
 F 1 "+12V" H 2550 3940 50  0000 C CNN
 F 2 "" H 2550 3800 50  0000 C CNN
@@
 VCC_12V
 $Comp
-L +12V #PWR?
+L +12V #PWR0107
 U 1 1 575C0189
 P 1650 800
-F 0 "#PWR?" H 1650 650 50  0001 C CNN
+F 0 "#PWR0107" H 1650 650 50  0001 C CNN
 F 1 "+12V" H 1650 940 50  0000 C CNN
 F 2 "" H 1650 800 50  0000 C CNN
@@
 	1650 900  1650 800
 $Comp
-L GND #PWR?
+L GND #PWR0108
 U 1 1 57662DD2
 P 4250 3700
-F 0 "#PWR?" H 4250 3450 50  0001 C CNN
+F 0 "#PWR0108" H 4250 3450 50  0001 C CNN
 F 1 "GND" H 4250 3550 50  0000 C CNN
 F 2 "" H 4250 3700 50  0000 C CNN
