File: board/evm/circuit/keyboard_blk_fpga.sch (KiCad schematic (older format))
At the start: 18 parts

Commit message: working on drc
Parts:
- gave numbers to parts that had none: 18
Connections:
- no-connect marks 1 -> 20

Commit message: working on footprint
Parts:
- C1, C4: footprint (none) -> Capacitors_SMD:C_0805
- C10, C11, C12, C13, C2, C3, C5, C6, C7, C8, C9: footprint (none) -> Capacitors_SMD:C_0402
- R5: footprint (none) -> Resistors_SMD:R_0402
- U5: footprint (none) -> TO_SOT_Packages_SMD:SOT-223
- U6: footprint (none) -> Housings_QFP:LQFP-100_14x14mm_Pitch0.5mm
Changed lines of the file:
@@
 F 0 "X1" H 3200 4150 50  0000 C CNN
 F 1 "IQXO/7X" H 3200 3850 50  0000 C CNN
-F 2 "" H 3200 3850 50  0000 C CNN
+F 2 "" H 3200 3850 50  0001 C CNN
 F 3 "" H 3200 3850 50  0000 C CNN
 	1    3200 3850
@@
 F 0 "U6" H 6700 4100 60  0000 C CNN
 F 1 "A3P060" H 6700 3900 60  0000 C CNN
-F 2 "" H 6350 4400 60  0000 C CNN
+F 2 "Housings_QFP:LQFP-100_14x14mm_Pitch0.5mm" H 6350 4400 60  0001 C CNN
 F 3 "" H 6350 4400 60  0000 C CNN
 	1    6750 3950
@@
 F 0 "J1" H 10150 5850 60  0000 C CNN
 F 1 "TagConnect" H 10650 5850 60  0000 C CNN
-F 2 "" H 10300 6050 60  0000 C CNN
+F 2 "" H 10300 6050 60  0001 C CNN
 F 3 "" H 10300 6050 60  0000 C CNN
 	1    10450 6000
@@
 F 0 "R5" V 9080 5150 50  0000 C CNN
 F 1 "R0" V 9000 5150 50  0000 C CNN
-F 2 "" V 8930 5150 50  0000 C CNN
+F 2 "Resistors_SMD:R_0402" V 8930 5150 50  0001 C CNN
 F 3 "" H 9000 5150 50  0000 C CNN
 	1    9000 5150
@@
 F 0 "U5" H 3250 7000 50  0000 C CNN
 F 1 "AP1117-1.5" H 3150 7500 50  0000 C CNN
-F 2 "" H 3150 7250 50  0000 C CNN
+F 2 "TO_SOT_Packages_SMD:SOT-223" H 3150 7250 50  0001 C CNN
 F 3 "" H 3150 7250 50  0000 C CNN
 	1    3150 7250
@@
 F 0 "C3" H 3660 7520 50  0000 L CNN
 F 1 "C_0.1uF" H 3660 7370 50  0000 L CNN
-F 2 "" H 3650 7450 50  0000 C CNN
+F 2 "Capacitors_SMD:C_0402" H 3650 7450 50  0001 C CNN
 F 3 "" H 3650 7450 50  0000 C CNN
 	1    3650 7450
@@
 F 0 "C2" H 2660 7520 50  0000 L CNN
 F 1 "C_0.1uF" H 2660 7370 50  0000 L CNN
-F 2 "" H 2650 7450 50  0000 C CNN
+F 2 "Capacitors_SMD:C_0402" H 2650 7450 50  0001 C CNN
 F 3 "" H 2650 7450 50  0000 C CNN
 	1    2650 7450
@@
 F 0 "C4" H 4010 7520 50  0000 L CNN
 F 1 "C_10uF" H 4010 7370 50  0000 L CNN
-F 2 "" H 4000 7450 50  0000 C CNN
+F 2 "Capacitors_SMD:C_0805" H 4000 7450 50  0001 C CNN
 F 3 "" H 4000 7450 50  0000 C CNN
 	1    4000 7450
@@
 F 0 "C1" H 2360 7520 50  0000 L CNN
 F 1 "C_10uF" H 2360 7370 50  0000 L CNN
-F 2 "" H 2350 7450 50  0000 C CNN
+F 2 "Capacitors_SMD:C_0805" H 2350 7450 50  0001 C CNN
 F 3 "" H 2350 7450 50  0000 C CNN
 	1    2350 7450
@@
 F 0 "C5" H 5510 7620 50  0000 L CNN
 F 1 "C_0.1uF" H 5510 7470 50  0000 L CNN
-F 2 "" H 5500 7550 50  0000 C CNN
+F 2 "Capacitors_SMD:C_0402" H 5500 7550 50  0001 C CNN
 F 3 "" H 5500 7550 50  0000 C CNN
 	1    5500 7550
@@
 F 0 "C7" H 5910 7620 50  0000 L CNN
 F 1 "C_0.1uF" H 5910 7470 50  0000 L CNN
-F 2 "" H 5900 7550 50  0000 C CNN
+F 2 "Capacitors_SMD:C_0402" H 5900 7550 50  0001 C CNN
 F 3 "" H 5900 7550 50  0000 C CNN
 	1    5900 7550
@@
 F 0 "C9" H 6310 7620 50  0000 L CNN
 F 1 "C_0.1uF" H 6310 7470 50  0000 L CNN
-F 2 "" H 6300 7550 50  0000 C CNN
+F 2 "Capacitors_SMD:C_0402" H 6300 7550 50  0001 C CNN
 F 3 "" H 6300 7550 50  0000 C CNN
 	1    6300 7550
@@
 F 0 "C11" H 6710 7620 50  0000 L CNN
 F 1 "C_0.1uF" H 6710 7470 50  0000 L CNN
-F 2 "" H 6700 7550 50  0000 C CNN
+F 2 "Capacitors_SMD:C_0402" H 6700 7550 50  0001 C CNN
 F 3 "" H 6700 7550 50  0000 C CNN
 	1    6700 7550
@@
 F 0 "C13" H 7110 7620 50  0000 L CNN
 F 1 "C_0.1uF" H 7110 7470 50  0000 L CNN
-F 2 "" H 7100 7550 50  0000 C CNN
+F 2 "Capacitors_SMD:C_0402" H 7100 7550 50  0001 C CNN
 F 3 "" H 7100 7550 50  0000 C CNN
 	1    7100 7550
@@
 F 0 "C6" H 5510 8570 50  0000 L CNN
 F 1 "C_0.1uF" H 5510 8420 50  0000 L CNN
-F 2 "" H 5500 8500 50  0000 C CNN
+F 2 "Capacitors_SMD:C_0402" H 5500 8500 50  0001 C CNN
 F 3 "" H 5500 8500 50  0000 C CNN
 	1    5500 8500
@@
 F 0 "C8" H 5910 8570 50  0000 L CNN
 F 1 "C_0.1uF" H 5910 8420 50  0000 L CNN
-F 2 "" H 5900 8500 50  0000 C CNN
+F 2 "Capacitors_SMD:C_0402" H 5900 8500 50  0001 C CNN
 F 3 "" H 5900 8500 50  0000 C CNN
 	1    5900 8500
@@
 F 0 "C10" H 6310 8570 50  0000 L CNN
 F 1 "C_0.1uF" H 6310 8420 50  0000 L CNN
-F 2 "" H 6300 8500 50  0000 C CNN
+F 2 "Capacitors_SMD:C_0402" H 6300 8500 50  0001 C CNN
 F 3 "" H 6300 8500 50  0000 C CNN
 	1    6300 8500
@@
 F 0 "C12" H 6710 8570 50  0000 L CNN
 F 1 "C_0.1uF" H 6710 8420 50  0000 L CNN
-F 2 "" H 6700 8500 50  0000 C CNN
+F 2 "Capacitors_SMD:C_0402" H 6700 8500 50  0001 C CNN
 F 3 "" H 6700 8500 50  0000 C CNN
 	1    6700 8500
