File: board/evm/circuit/oh-my-keyboard.sch (KiCad schematic (older format))
At the start: 39 parts

Commit message: working on drc
Parts:
- gave numbers to parts that had none: 39
Connections:
- no-connect marks 6 -> 20
Other:
- moved on the sheet: W34

Commit message: working on footprint
Parts:
- R2: footprint (none) -> Resistors_SMD:R_0402
- W1, W10, W11, W12, W13, W14, W15, W16, W17, W18, W19, W2, W20, W21, W22, W23, W24, W25, W26, W27, W28, W29, W3, W30, W31, W32, W33, W34, W35, W36, W4, W5, W6, W7, W8, W9: footprint (none) -> Connect:PINTST
Changed lines of the file:
@@
 F 0 "P1" H 12950 6150 50  0000 C CNN
 F 1 "CONN_02X12" V 12950 5500 50  0000 C CNN
-F 2 "" H 12950 4300 50  0000 C CNN
+F 2 "" H 12950 4300 50  0001 C CNN
 F 3 "" H 12950 4300 50  0000 C CNN
 	1    12950 5500
@@
 F 0 "R1" V 7880 6900 50  0000 C CNN
 F 1 "Photores" V 8010 6900 50  0000 C TNN
-F 2 "" V 7730 6900 50  0000 C CNN
+F 2 "" V 7730 6900 50  0001 C CNN
 F 3 "" H 7800 6900 50  0000 C CNN
 	1    7800 6900
@@
 F 0 "R2" V 8130 6450 50  0000 C CNN
 F 1 "R62K" V 8050 6450 50  0000 C CNN
-F 2 "" V 7980 6450 50  0000 C CNN
+F 2 "Resistors_SMD:R_0402" V 7980 6450 50  0001 C CNN
 F 3 "" H 8050 6450 50  0000 C CNN
 	1    8050 6450
@@
 F 0 "W20" H 6900 4270 50  0000 C CNN
 F 1 "TP" H 6900 4200 50  0000 C CNN
-F 2 "" H 7100 4000 50  0000 C CNN
+F 2 "Connect:PINTST" H 7100 4000 50  0001 C CNN
 F 3 "" H 7100 4000 50  0000 C CNN
 	1    6900 4000
@@
 F 0 "W3" H 6750 4170 50  0000 C CNN
 F 1 "TP" H 6750 4100 50  0000 C CNN
-F 2 "" H 6950 3900 50  0000 C CNN
+F 2 "Connect:PINTST" H 6950 3900 50  0001 C CNN
 F 3 "" H 6950 3900 50  0000 C CNN
 	1    6750 3900
@@
 F 0 "W4" H 6750 4420 50  0000 C CNN
 F 1 "TP" H 6750 4350 50  0000 C CNN
-F 2 "" H 6950 4150 50  0000 C CNN
+F 2 "Connect:PINTST" H 6950 4150 50  0001 C CNN
 F 3 "" H 6950 4150 50  0000 C CNN
 	1    6750 4150
@@
 F 0 "W21" H 6900 4520 50  0000 C CNN
 F 1 "TP" H 6900 4450 50  0000 C CNN
-F 2 "" H 7100 4250 50  0000 C CNN
+F 2 "Connect:PINTST" H 7100 4250 50  0001 C CNN
 F 3 "" H 7100 4250 50  0000 C CNN
 	1    6900 4250
@@
 F 0 "W5" H 6750 4670 50  0000 C CNN
 F 1 "TP" H 6750 4600 50  0000 C CNN
-F 2 "" H 6950 4400 50  0000 C CNN
+F 2 "Connect:PINTST" H 6950 4400 50  0001 C CNN
 F 3 "" H 6950 4400 50  0000 C CNN
 	1    6750 4400
@@
 F 0 "W22" H 6900 4770 50  0000 C CNN
 F 1 "TP" H 6900 4700 50  0000 C CNN
-F 2 "" H 7100 4500 50  0000 C CNN
+F 2 "Connect:PINTST" H 7100 4500 50  0001 C CNN
 F 3 "" H 7100 4500 50  0000 C CNN
 	1    6900 4500
@@
 F 0 "W6" H 6750 4920 50  0000 C CNN
 F 1 "TP" H 6750 4850 50  0000 C CNN
-F 2 "" H 6950 4650 50  0000 C CNN
+F 2 "Connect:PINTST" H 6950 4650 50  0001 C CNN
 F 3 "" H 6950 4650 50  0000 C CNN
 	1    6750 4650
@@
 F 0 "W23" H 6900 5020 50  0000 C CNN
 F 1 "TP" H 6900 4950 50  0000 C CNN
-F 2 "" H 7100 4750 50  0000 C CNN
+F 2 "Connect:PINTST" H 7100 4750 50  0001 C CNN
 F 3 "" H 7100 4750 50  0000 C CNN
 	1    6900 4750
@@
 F 0 "W7" H 6750 5170 50  0000 C CNN
 F 1 "TP" H 6750 5100 50  0000 C CNN
-F 2 "" H 6950 4900 50  0000 C CNN
+F 2 "Connect:PINTST" H 6950 4900 50  0001 C CNN
 F 3 "" H 6950 4900 50  0000 C CNN
 	1    6750 4900
@@
 F 0 "W14" H 6850 5270 50  0000 C CNN
 F 1 "TP" H 6850 5200 50  0000 C CNN
-F 2 "" H 7050 5000 50  0000 C CNN
+F 2 "Connect:PINTST" H 7050 5000 50  0001 C CNN
 F 3 "" H 7050 5000 50  0000 C CNN
 	1    6850 5000
@@
 F 0 "W8" H 6750 5370 50  0000 C CNN
 F 1 "TP" H 6750 5300 50  0000 C CNN
-F 2 "" H 6950 5100 50  0000 C CNN
+F 2 "Connect:PINTST" H 6950 5100 50  0001 C CNN
 F 3 "" H 6950 5100 50  0000 C CNN
 	1    6750 5100
@@
 F 0 "W15" H 6850 5470 50  0000 C CNN
 F 1 "TP" H 6850 5400 50  0000 C CNN
-F 2 "" H 7050 5200 50  0000 C CNN
+F 2 "Connect:PINTST" H 7050 5200 50  0001 C CNN
 F 3 "" H 7050 5200 50  0000 C CNN
 	1    6850 5200
@@
 F 0 "W9" H 6750 5620 50  0000 C CNN
 F 1 "TP" H 6750 5550 50  0000 C CNN
-F 2 "" H 6950 5350 50  0000 C CNN
+F 2 "Connect:PINTST" H 6950 5350 50  0001 C CNN
 F 3 "" H 6950 5350 50  0000 C CNN
 	1    6750 5350
@@
 F 0 "W16" H 6850 5720 50  0000 C CNN
 F 1 "TP" H 6850 5650 50  0000 C CNN
-F 2 "" H 7050 5450 50  0000 C CNN
+F 2 "Connect:PINTST" H 7050 5450 50  0001 C CNN
 F 3 "" H 7050 5450 50  0000 C CNN
 	1    6850 5450
@@
 F 0 "W10" H 6750 5820 50  0000 C CNN
 F 1 "TP" H 6750 5750 50  0000 C CNN
-F 2 "" H 6950 5550 50  0000 C CNN
+F 2 "Connect:PINTST" H 6950 5550 50  0001 C CNN
 F 3 "" H 6950 5550 50  0000 C CNN
 	1    6750 5550
@@
 F 0 "W17" H 6850 5920 50  0000 C CNN
 F 1 "TP" H 6850 5850 50  0000 C CNN
-F 2 "" H 7050 5650 50  0000 C CNN
+F 2 "Connect:PINTST" H 7050 5650 50  0001 C CNN
 F 3 "" H 7050 5650 50  0000 C CNN
 	1    6850 5650
@@
 F 0 "W11" H 6750 6020 50  0000 C CNN
 F 1 "TP" H 6750 5950 50  0000 C CNN
-F 2 "" H 6950 5750 50  0000 C CNN
+F 2 "Connect:PINTST" H 6950 5750 50  0001 C CNN
 F 3 "" H 6950 5750 50  0000 C CNN
 	1    6750 5750
@@
 F 0 "W18" H 6850 6120 50  0000 C CNN
 F 1 "TP" H 6850 6050 50  0000 C CNN
-F 2 "" H 7050 5850 50  0000 C CNN
+F 2 "Connect:PINTST" H 7050 5850 50  0001 C CNN
 F 3 "" H 7050 5850 50  0000 C CNN
 	1    6850 5850
@@
 F 0 "W12" H 6750 6220 50  0000 C CNN
 F 1 "TP" H 6750 6150 50  0000 C CNN
-F 2 "" H 6950 5950 50  0000 C CNN
+F 2 "Connect:PINTST" H 6950 5950 50  0001 C CNN
 F 3 "" H 6950 5950 50  0000 C CNN
 	1    6750 5950
@@
 F 0 "W19" H 6850 6320 50  0000 C CNN
 F 1 "TP" H 6850 6250 50  0000 C CNN
-F 2 "" H 7050 6050 50  0000 C CNN
+F 2 "Connect:PINTST" H 7050 6050 50  0001 C CNN
 F 3 "" H 7050 6050 50  0000 C CNN
 	1    6850 6050
@@
 F 0 "W13" H 6800 6720 50  0000 C CNN
 F 1 "TP" H 6800 6650 50  0000 C CNN
-F 2 "" H 7000 6450 50  0000 C CNN
+F 2 "Connect:PINTST" H 7000 6450 50  0001 C CNN
 F 3 "" H 7000 6450 50  0000 C CNN
 	1    6800 6450
@@
 F 0 "W25" H 7550 2070 50  0000 C CNN
 F 1 "TP" H 7550 2000 50  0000 C CNN
-F 2 "" H 7750 1800 50  0000 C CNN
+F 2 "Connect:PINTST" H 7750 1800 50  0001 C CNN
 F 3 "" H 7750 1800 50  0000 C CNN
 	1    7550 1800
@@
 F 0 "W24" H 7500 2170 50  0000 C CNN
 F 1 "TP" H 7500 2100 50  0000 C CNN
-F 2 "" H 7700 1900 50  0000 C CNN
+F 2 "Connect:PINTST" H 7700 1900 50  0001 C CNN
 F 3 "" H 7700 1900 50  0000 C CNN
 	1    7500 1900
@@
 F 0 "W28" H 7950 2270 50  0000 C CNN
 F 1 "TP" H 7950 2200 50  0000 C CNN
-F 2 "" H 8150 2000 50  0000 C CNN
+F 2 "Connect:PINTST" H 8150 2000 50  0001 C CNN
 F 3 "" H 8150 2000 50  0000 C CNN
 	1    7950 2000
@@
 F 0 "W26" H 7550 3120 50  0000 C CNN
 F 1 "TP" H 7550 3050 50  0000 C CNN
-F 2 "" H 7750 2850 50  0000 C CNN
+F 2 "Connect:PINTST" H 7750 2850 50  0001 C CNN
 F 3 "" H 7750 2850 50  0000 C CNN
 	1    7550 2850
@@
 F 0 "W27" H 7550 3220 50  0000 C CNN
 F 1 "TP" H 7550 3150 50  0000 C CNN
-F 2 "" H 7750 2950 50  0000 C CNN
+F 2 "Connect:PINTST" H 7750 2950 50  0001 C CNN
 F 3 "" H 7750 2950 50  0000 C CNN
 	1    7550 2950
@@
 F 0 "W30" H 11150 2970 50  0000 C CNN
 F 1 "TP" H 11150 2900 50  0000 C CNN
-F 2 "" H 11350 2700 50  0000 C CNN
+F 2 "Connect:PINTST" H 11350 2700 50  0001 C CNN
 F 3 "" H 11350 2700 50  0000 C CNN
 	1    11150 2700
@@
 F 0 "W33" H 11250 3070 50  0000 C CNN
 F 1 "TP" H 11250 3000 50  0000 C CNN
-F 2 "" H 11450 2800 50  0000 C CNN
+F 2 "Connect:PINTST" H 11450 2800 50  0001 C CNN
 F 3 "" H 11450 2800 50  0000 C CNN
 	1    11250 2800
@@
 F 0 "W35" H 11350 3170 50  0000 C CNN
 F 1 "TP" H 11350 3100 50  0000 C CNN
-F 2 "" H 11550 2900 50  0000 C CNN
+F 2 "Connect:PINTST" H 11550 2900 50  0001 C CNN
 F 3 "" H 11550 2900 50  0000 C CNN
 	1    11350 2900
@@
 F 0 "W31" H 11150 3270 50  0000 C CNN
 F 1 "TP" H 11150 3200 50  0000 C CNN
-F 2 "" H 11350 3000 50  0000 C CNN
+F 2 "Connect:PINTST" H 11350 3000 50  0001 C CNN
 F 3 "" H 11350 3000 50  0000 C CNN
 	1    11150 3000
@@
 F 0 "W34" H 11250 3370 50  0000 C CNN
 F 1 "TP" H 11250 3300 50  0000 C CNN
-F 2 "" H 11450 3100 50  0000 C CNN
+F 2 "Connect:PINTST" H 11450 3100 50  0001 C CNN
 F 3 "" H 11450 3100 50  0000 C CNN
 	1    11250 3100
@@
 F 0 "W29" H 11050 3470 50  0000 C CNN
 F 1 "TP" H 11050 3400 50  0000 C CNN
-F 2 "" H 11250 3200 50  0000 C CNN
+F 2 "Connect:PINTST" H 11250 3200 50  0001 C CNN
 F 3 "" H 11250 3200 50  0000 C CNN
 	1    11050 3200
@@
 F 0 "W32" H 11150 3570 50  0000 C CNN
 F 1 "TP" H 11150 3500 50  0000 C CNN
-F 2 "" H 11350 3300 50  0000 C CNN
+F 2 "Connect:PINTST" H 11350 3300 50  0001 C CNN
 F 3 "" H 11350 3300 50  0000 C CNN
 	1    11150 3300
@@
 F 0 "W36" H 11400 4070 50  0000 C CNN
 F 1 "TP" H 11400 4000 50  0000 C CNN
-F 2 "" H 11600 3800 50  0000 C CNN
+F 2 "Connect:PINTST" H 11600 3800 50  0001 C CNN
 F 3 "" H 11600 3800 50  0000 C CNN
 	1    11400 3800
@@
 F 0 "W1" H 1650 6570 50  0000 C CNN
 F 1 "TP" H 1650 6500 50  0000 C CNN
-F 2 "" H 1850 6300 50  0000 C CNN
+F 2 "Connect:PINTST" H 1850 6300 50  0001 C CNN
 F 3 "" H 1850 6300 50  0000 C CNN
 	1    1650 6300
@@
 F 0 "W2" H 2000 6520 50  0000 C CNN
 F 1 "TP" H 2000 6450 50  0000 C CNN
-F 2 "" H 2200 6250 50  0000 C CNN
+F 2 "Connect:PINTST" H 2200 6250 50  0001 C CNN
 F 3 "" H 2200 6250 50  0000 C CNN
 	1    2000 6250
